File: SpaceCadet.kicad_sch (KiCad schematic)
At the start: 35 parts, among them J0 Conn_02x17_Odd_Even, J3_1 Conn_01x04, J3_2 Conn_01x04, U1 74LS154, U2 8048, Y3 Crystal 3.58MHz

Commit message: Added traces, jumpers to front to use DRC. Fixed lots of real and imaginary DRC errors/warnings.
Other:
- moved on the sheet: JP25
Changed lines of the file:
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@@
   (junction (at 53.34 80.645) (diameter 0) (color 0 0 0 0)
   )
-  (junction (at 178.435 107.95) (diameter 0) (color 0 0 0 0)
-  )
   (junction (at 120.65 107.95) (diameter 0) (color 0 0 0 0)
   )
@@
   )
   (junction (at 193.675 105.41) (diameter 0) (color 0 0 0 0)
+  )
+  (junction (at 178.435 105.41) (diameter 0) (color 0 0 0 0)
   )
   (junction (at 178.435 101.6) (diameter 0) (color 0 0 0 0)
@@
     (stroke (width 0) (type default) (color 0 0 0 0))
   )
+  (wire (pts (xy 178.435 105.41) (xy 178.435 110.49))
+    (stroke (width 0) (type default) (color 0 0 0 0))
+  )
   (wire (pts (xy 199.39 51.435) (xy 203.2 51.435))
     (stroke (width 0) (type default) (color 0 0 0 0))
@@
     (stroke (width 0) (type default) (color 0 0 0 0))
   )
-  (wire (pts (xy 175.895 107.95) (xy 178.435 107.95))
+  (wire (pts (xy 175.895 105.41) (xy 178.435 105.41))
     (stroke (width 0) (type default) (color 0 0 0 0))
   )
@@
     (stroke (width 0) (type default) (color 0 0 0 0))
   )
+  (wire (pts (xy 175.895 105.41) (xy 175.895 110.49))
+    (stroke (width 0) (type default) (color 0 0 0 0))
+  )
   (bus (pts (xy 183.515 133.985) (xy 183.515 135.255))
     (stroke (width 0) (type default) (color 0 0 0 0))
@@
     (stroke (width 0) (type default) (color 0 0 0 0))
   )
+  (wire (pts (xy 178.435 101.6) (xy 178.435 105.41))
+    (stroke (width 0) (type default) (color 0 0 0 0))
+  )
   (wire (pts (xy 199.39 40.005) (xy 203.2 40.005))
     (stroke (width 0) (type default) (color 0 0 0 0))
@@
     (stroke (width 0) (type default) (color 0 0 0 0))
   )
-  (wire (pts (xy 175.895 110.49) (xy 175.895 107.95))
-    (stroke (width 0) (type default) (color 0 0 0 0))
-  )
   (wire (pts (xy 66.675 42.545) (xy 74.93 42.545))
     (stroke (width 0) (type default) (color 0 0 0 0))
@@
     (stroke (width 0) (type default) (color 0 0 0 0))
   )
-  (wire (pts (xy 178.435 107.95) (xy 178.435 110.49))
-    (stroke (width 0) (type default) (color 0 0 0 0))
-  )
   (bus (pts (xy 59.055 137.16) (xy 59.055 134.62))
     (stroke (width 0) (type default) (color 0 0 0 0))
@@
   )
   (polyline (pts (xy 228.6 19.685) (xy 228.6 115.57))
-    (stroke (width 0) (type default) (color 0 0 0 0))
-  )
-  (wire (pts (xy 178.435 101.6) (xy 178.435 107.95))
     (stroke (width 0) (type default) (color 0 0 0 0))
   )
@@
     (effects (font (size 1.27 1.27)) (justify left bottom))
   )
+  (label "GND" (at 188.595 110.49 90)
+    (effects (font (size 1.27 1.27)) (justify left bottom))
+  )
   (label "COL7" (at 95.25 152.4 0) (fields_autoplaced)
     (effects (font (size 1.27 1.27)) (justify left bottom))
@@
   )
   (label "ROW1" (at 68.58 65.405 0) (fields_autoplaced)
+    (effects (font (size 1.27 1.27)) (justify left bottom))
+  )
+  (label "+5V" (at 178.435 110.49 90)
     (effects (font (size 1.27 1.27)) (justify left bottom))
   )
@@
   (symbol (lib_id "Jumper:Jumper_2_Bridged") (at 208.28 62.865 0) (unit 1)
     (in_bom yes) (on_board yes)
-    (property "Reference" "JP24" (id 0) (at 208.28 61.595 0))
+    (property "Reference" "JP24" (id 0) (at 208.28 64.77 0))
     (property "Value" "Jumper Bridged" (id 1) (at 191.135 62.865 0)
       (effects (font (size 1.27 1.27)) (justify right))
@@
   (symbol (lib_id "Jumper:Jumper_2_Open") (at 260.35 92.71 0) (unit 1)
     (in_bom yes) (on_board yes)
-    (property "Reference" "JP29" (id 0) (at 262.255 93.98 0)
-      (effects (font (size 1.27 1.27)) (justify right))
-    )
+    (property "Reference" "JP29" (id 0) (at 260.35 94.615 0))
     (property "Value" "Jumper Open" (id 1) (at 243.205 92.71 0)
       (effects (font (size 1.27 1.27)) (justify right))
@@
   (symbol (lib_id "Jumper:Jumper_2_Bridged") (at 208.28 40.005 0) (unit 1)
     (in_bom yes) (on_board yes)
-    (property "Reference" "JP20" (id 0) (at 208.28 38.735 0))
+    (property "Reference" "JP20" (id 0) (at 208.28 41.91 0))
     (property "Value" "Jumper Bridged" (id 1) (at 191.135 40.005 0)
       (effects (font (size 1.27 1.27)) (justify right))
@@
   (symbol (lib_id "Jumper:Jumper_2_Open") (at 260.35 104.14 0) (unit 1)
     (in_bom yes) (on_board yes)
-    (property "Reference" "JP31" (id 0) (at 262.255 105.41 0)
-      (effects (font (size 1.27 1.27)) (justify right))
-    )
+    (property "Reference" "JP31" (id 0) (at 260.35 106.045 0))
     (property "Value" "Jumper Open" (id 1) (at 243.205 104.14 0)
       (effects (font (size 1.27 1.27)) (justify right))
@@
   (symbol (lib_id "Jumper:Jumper_2_Open") (at 260.35 109.855 0) (unit 1)
     (in_bom yes) (on_board yes)
-    (property "Reference" "JP32" (id 0) (at 262.255 111.125 0)
-      (effects (font (size 1.27 1.27)) (justify right))
-    )
+    (property "Reference" "JP32" (id 0) (at 260.35 111.76 0))
     (property "Value" "Jumper Open" (id 1) (at 243.205 109.855 0)
       (effects (font (size 1.27 1.27)) (justify right))
@@
   (symbol (lib_id "Jumper:Jumper_2_Open") (at 260.35 98.425 0) (unit 1)
     (in_bom yes) (on_board yes)
-    (property "Reference" "JP30" (id 0) (at 262.255 99.695 0)
-      (effects (font (size 1.27 1.27)) (justify right))
-    )
+    (property "Reference" "JP30" (id 0) (at 260.35 100.33 0))
     (property "Value" "Jumper Open" (id 1) (at 243.205 98.425 0)
       (effects (font (size 1.27 1.27)) (justify right))
@@
   (symbol (lib_id "Jumper:Jumper_2_Open") (at 260.35 75.565 0) (unit 1)
     (in_bom yes) (on_board yes)
-    (property "Reference" "JP26" (id 0) (at 262.255 76.835 0)
-      (effects (font (size 1.27 1.27)) (justify right))
-    )
+    (property "Reference" "JP26" (id 0) (at 260.35 77.47 0))
     (property "Value" "Jumper Open" (id 1) (at 243.205 75.565 0)
       (effects (font (size 1.27 1.27)) (justify right))
@@
     (pin "2")
   )
-  (symbol (lib_id "Jumper:Jumper_2_Open") (at 260.35 69.85 0) (mirror x) (unit 1)
-    (in_bom yes) (on_board yes)
-    (property "Reference" "JP25" (id 0) (at 262.89 67.945 0)
-      (effects (font (size 1.27 1.27)) (justify right))
-    )
+  (symbol (lib_id "Jumper:Jumper_2_Open") (at 260.35 69.85 0) (unit 1)
+    (in_bom yes) (on_board yes)
+    (property "Reference" "JP25" (id 0) (at 260.35 71.755 0))
     (property "Value" "Jumper Open" (id 1) (at 243.205 69.85 0)
       (effects (font (size 1.27 1.27)) (justify right))
@@
   (symbol (lib_id "Jumper:Jumper_2_Open") (at 260.35 34.29 0) (unit 1)
     (in_bom yes) (on_board yes)
-    (property "Reference" "JP19" (id 0) (at 262.255 31.75 0)
-      (effects (font (size 1.27 1.27)) (justify right))
-    )
+    (property "Reference" "JP19" (id 0) (at 260.35 36.195 0))
     (property "Value" "Jumper Open" (id 1) (at 243.205 34.29 0)
       (effects (font (size 1.27 1.27)) (justify right))
@@
   (symbol (lib_id "Jumper:Jumper_2_Open") (at 260.35 28.575 0) (unit 1)
     (in_bom yes) (on_board yes)
-    (property "Reference" "JP18" (id 0) (at 262.255 26.035 0)
-      (effects (font (size 1.27 1.27)) (justify right))
-    )
+    (property "Reference" "JP18" (id 0) (at 260.35 30.48 0))
     (property "Value" "Jumper Open" (id 1) (at 243.205 28.575 0)
       (effects (font (size 1.27 1.27)) (justify right))
@@
   (symbol (lib_id "Jumper:Jumper_2_Open") (at 260.35 57.15 0) (unit 1)
     (in_bom yes) (on_board yes)
-    (property "Reference" "JP23" (id 0) (at 262.255 54.61 0)
-      (effects (font (size 1.27 1.27)) (justify right))
-    )
+    (property "Reference" "JP23" (id 0) (at 260.35 59.055 0))
     (property "Value" "Jumper Open" (id 1) (at 243.205 57.15 0)
       (effects (font (size 1.27 1.27)) (justify right))
@@
   (symbol (lib_id "Jumper:Jumper_2_Bridged") (at 208.28 45.72 0) (unit 1)
     (in_bom yes) (on_board yes)
-    (property "Reference" "JP21" (id 0) (at 208.28 44.45 0))
+    (property "Reference" "JP21" (id 0) (at 208.28 47.625 0))
     (property "Value" "Jumper Bridged" (id 1) (at 191.135 45.72 0)
       (effects (font (size 1.27 1.27)) (justify right))
@@
   (symbol (lib_id "Jumper:Jumper_2_Open") (at 260.35 86.995 0) (unit 1)
     (in_bom yes) (on_board yes)
-    (property "Reference" "JP28" (id 0) (at 262.255 88.265 0)
-      (effects (font (size 1.27 1.27)) (justify right))
-    )
+    (property "Reference" "JP28" (id 0) (at 260.35 88.9 0))
     (property "Value" "Jumper Open" (id 1) (at 243.205 86.995 0)
       (effects (font (size 1.27 1.27)) (justify right))
@@
   (symbol (lib_id "Jumper:Jumper_2_Bridged") (at 208.28 51.435 0) (unit 1)
     (in_bom yes) (on_board yes)
-    (property "Reference" "JP22" (id 0) (at 208.28 50.165 0))
+    (property "Reference" "JP22" (id 0) (at 208.28 53.34 0))
     (property "Value" "Jumper Bridged" (id 1) (at 191.135 51.435 0)
       (effects (font (size 1.27 1.27)) (justify right))
@@
   (symbol (lib_id "Jumper:Jumper_2_Open") (at 260.35 81.28 0) (unit 1)
     (in_bom yes) (on_board yes)
-    (property "Reference" "JP27" (id 0) (at 262.255 82.55 0)
-      (effects (font (size 1.27 1.27)) (justify right))
-    )
+    (property "Reference" "JP27" (id 0) (at 260.35 83.185 0))
     (property "Value" "Jumper Open" (id 1) (at 243.205 81.28 0)
       (effects (font (size 1.27 1.27)) (justify right))
@@
       (reference "#PWR0113") (unit 1) (value "+5V") (footprint "")
     )
+    (path "/1a8342a5-15fc-454c-84eb-2b470c08f569/44de499e-d74e-4a0b-ad44-b5559c965905"
+      (reference "#PWR0114") (unit 1) (value "+5V") (footprint "")
+    )
     (path "/4b693529-fe06-44af-a160-67a5ffd8665d"
