File: SpaceCadet.kicad_sch (KiCad schematic)
At the start: 35 parts, among them J0 Conn_02x17_Odd_Even, J3_1 Conn_01x04, J3_2 Conn_01x04, U1 74LS154, U2 8048, Y3 Crystal 3.58MHz

Commit message: Added front-side copper for constraint check. Debugged switch footprint.
Parts:
- C12, C13, C14, C15, Y3: footprint (none) -> TestPoint:Two_Pad_Through_Hole_10.4mm
- C16: footprint (none) -> TestPoint:Two_Pad_Through_Hole_20mm
- C17: footprint (none) -> TestPoint:Two_Pad_Through_Hole_12mm
- R10, R11, R4, R5, R6, R7, R8, R9: footprint (none) -> TestPoint:Two_Pad_Through_Hole_12.4mm
Changed lines of the file:
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@@
     (property "Reference" "C16" (id 0) (at 181.61 95.25 90))
     (property "Value" "22uF 15v" (id 1) (at 191.135 95.25 90))
-    (property "Footprint" "" (id 2) (at 184.785 96.52 0)
+    (property "Footprint" "TestPoint:Two_Pad_Through_Hole_20mm" (id 2) (at 184.785 96.52 0)
       (effects (font (size 1.27 1.27)) hide)
     )
@@
     (property "Reference" "Y3" (id 0) (at 120.65 93.0275 0))
     (property "Value" "Crystal 3.58MHz" (id 1) (at 120.65 94.7897 0))
-    (property "Footprint" "" (id 2) (at 120.65 98.425 0)
+    (property "Footprint" "TestPoint:Two_Pad_Through_Hole_10.4mm" (id 2) (at 120.65 98.425 0)
       (effects (font (size 1.27 1.27)) hide)
     )
@@
     (property "Reference" "C12" (id 0) (at 88.9 120.015 90))
     (property "Value" "10pF" (id 1) (at 89.535 121.92 90))
-    (property "Footprint" "" (id 2) (at 89.535 122.2248 0)
+    (property "Footprint" "TestPoint:Two_Pad_Through_Hole_10.4mm" (id 2) (at 89.535 122.2248 0)
       (effects (font (size 1.27 1.27)) hide)
     )
@@
     (property "Reference" "C15" (id 0) (at 182.88 100.33 90))
     (property "Value" "15pF" (id 1) (at 182.245 102.87 90))
-    (property "Footprint" "" (id 2) (at 185.42 101.6 0)
+    (property "Footprint" "TestPoint:Two_Pad_Through_Hole_10.4mm" (id 2) (at 185.42 101.6 0)
       (effects (font (size 1.27 1.27)) hide)
     )
@@
     (property "Reference" "R4" (id 0) (at 50.8 95.25 90))
     (property "Value" "1K" (id 1) (at 50.165 86.36 90))
-    (property "Footprint" "" (id 2) (at 49.784 89.281 90)
+    (property "Footprint" "TestPoint:Two_Pad_Through_Hole_12.4mm" (id 2) (at 49.784 89.281 90)
       (effects (font (size 1.27 1.27)) hide)
     )
@@
     (property "Reference" "R10" (id 0) (at 38.1 95.25 90))
     (property "Value" "1K" (id 1) (at 37.465 86.36 90))
-    (property "Footprint" "" (id 2) (at 37.084 89.281 90)
+    (property "Footprint" "TestPoint:Two_Pad_Through_Hole_12.4mm" (id 2) (at 37.084 89.281 90)
       (effects (font (size 1.27 1.27)) hide)
     )
@@
     (property "Reference" "R6" (id 0) (at 48.26 95.25 90))
     (property "Value" "1K" (id 1) (at 47.625 86.36 90))
-    (property "Footprint" "" (id 2) (at 47.244 89.281 90)
+    (property "Footprint" "TestPoint:Two_Pad_Through_Hole_12.4mm" (id 2) (at 47.244 89.281 90)
       (effects (font (size 1.27 1.27)) hide)
     )
@@
     (property "Reference" "R5" (id 0) (at 53.34 95.25 90))
     (property "Value" "1K" (id 1) (at 52.705 86.36 90))
-    (property "Footprint" "" (id 2) (at 52.324 89.281 90)
+    (property "Footprint" "TestPoint:Two_Pad_Through_Hole_12.4mm" (id 2) (at 52.324 89.281 90)
       (effects (font (size 1.27 1.27)) hide)
     )
@@
     (property "Reference" "R9" (id 0) (at 40.64 95.25 90))
     (property "Value" "1K" (id 1) (at 40.005 86.36 90))
-    (property "Footprint" "" (id 2) (at 39.624 89.281 90)
+    (property "Footprint" "TestPoint:Two_Pad_Through_Hole_12.4mm" (id 2) (at 39.624 89.281 90)
       (effects (font (size 1.27 1.27)) hide)
     )
@@
       (effects (font (size 1.27 1.27)) (justify left))
     )
-    (property "Footprint" "" (id 2) (at 115.9002 107.95 0)
+    (property "Footprint" "TestPoint:Two_Pad_Through_Hole_10.4mm" (id 2) (at 115.9002 107.95 0)
       (effects (font (size 1.27 1.27)) hide)
     )
@@
       (effects (font (size 1.27 1.27)) (justify left))
     )
-    (property "Footprint" "" (id 2) (at 127.3302 107.95 0)
+    (property "Footprint" "TestPoint:Two_Pad_Through_Hole_10.4mm" (id 2) (at 127.3302 107.95 0)
       (effects (font (size 1.27 1.27)) hide)
     )
@@
     (property "Reference" "C17" (id 0) (at 203.2 131.445 90))
     (property "Value" "4.7uF 25v" (id 1) (at 200.66 133.35 90))
-    (property "Footprint" "" (id 2) (at 199.39 130.175 0)
+    (property "Footprint" "TestPoint:Two_Pad_Through_Hole_12mm" (id 2) (at 199.39 130.175 0)
       (effects (font (size 1.27 1.27)) hide)
     )
@@
     (property "Reference" "R7" (id 0) (at 45.72 95.25 90))
     (property "Value" "1K" (id 1) (at 45.085 86.36 90))
-    (property "Footprint" "" (id 2) (at 44.704 89.281 90)
+    (property "Footprint" "TestPoint:Two_Pad_Through_Hole_12.4mm" (id 2) (at 44.704 89.281 90)
       (effects (font (size 1.27 1.27)) hide)
     )
@@
     (property "Reference" "R11" (id 0) (at 35.56 95.25 90))
     (property "Value" "1K" (id 1) (at 34.925 86.36 90))
-    (property "Footprint" "" (id 2) (at 34.544 89.281 90)
+    (property "Footprint" "TestPoint:Two_Pad_Through_Hole_12.4mm" (id 2) (at 34.544 89.281 90)
       (effects (font (size 1.27 1.27)) hide)
     )
@@
     (property "Reference" "R8" (id 0) (at 43.18 95.25 90))
     (property "Value" "1K" (id 1) (at 42.545 86.36 90))
-    (property "Footprint" "" (id 2) (at 42.164 89.281 90)
+    (property "Footprint" "TestPoint:Two_Pad_Through_Hole_12.4mm" (id 2) (at 42.164 89.281 90)
       (effects (font (size 1.27 1.27)) hide)
     )
@@
     )
     (path "/4b693529-fe06-44af-a160-67a5ffd8665d"
-      (reference "C12") (unit 1) (value "10pF") (footprint "")
+      (reference "C12") (unit 1) (value "10pF") (footprint "TestPoint:Two_Pad_Through_Hole_10.4mm")
     )
     (path "/8cff2a90-9996-4fb8-b834-7ba83869fd3b"
-      (reference "C13") (unit 1) (value "10pF") (footprint "")
+      (reference "C13") (unit 1) (value "10pF") (footprint "TestPoint:Two_Pad_Through_Hole_10.4mm")
     )
     (path "/8579f6ff-d916-43cb-9f3a-9ef7b7dec6ac"
-      (reference "C14") (unit 1) (value "10pF") (footprint "")
+      (reference "C14") (unit 1) (value "10pF") (footprint "TestPoint:Two_Pad_Through_Hole_10.4mm")
     )
     (path "/4ec161d3-1c9b-4ea4-8ce3-cad9856a00a1"
-      (reference "C15") (unit 1) (value "15pF") (footprint "")
+      (reference "C15") (unit 1) (value "15pF") (footprint "TestPoint:Two_Pad_Through_Hole_10.4mm")
     )
     (path "/0483c138-e6fc-4834-bde0-ce6afaa0b50e"
-      (reference "C16") (unit 1) (value "22uF 15v") (footprint "")
+      (reference "C16") (unit 1) (value "22uF 15v") (footprint "TestPoint:Two_Pad_Through_Hole_20mm")
     )
     (path "/94b91b8a-0258-4cda-a957-e6f302c9f04e"
-      (reference "C17") (unit 1) (value "4.7uF 25v") (footprint "")
+      (reference "C17") (unit 1) (value "4.7uF 25v") (footprint "TestPoint:Two_Pad_Through_Hole_12mm")
     )
     (path "/1ea855f8-a5b1-424e-a642-dd01e460d8f4"
@@
     )
     (path "/4ed57943-0461-493e-8f46-26d1eea10a82"
-      (reference "R4") (unit 1) (value "1K") (footprint "")
+      (reference "R4") (unit 1) (value "1K") (footprint "TestPoint:Two_Pad_Through_Hole_12.4mm")
     )
     (path "/7ef65beb-8399-4097-ac13-2d05b63259d4"
-      (reference "R5") (unit 1) (value "1K") (footprint "")
+      (reference "R5") (unit 1) (value "1K") (footprint "TestPoint:Two_Pad_Through_Hole_12.4mm")
     )
     (path "/585e9c7f-d46a-4180-8342-4d9663c8f2cc"
-      (reference "R6") (unit 1) (value "1K") (footprint "")
+      (reference "R6") (unit 1) (value "1K") (footprint "TestPoint:Two_Pad_Through_Hole_12.4mm")
     )
     (path "/b1af4875-6c7a-4214-901c-5aeac72b67c9"
-      (reference "R7") (unit 1) (value "1K") (footprint "")
+      (reference "R7") (unit 1) (value "1K") (footprint "TestPoint:Two_Pad_Through_Hole_12.4mm")
     )
     (path "/e80dacb6-6a6c-44ed-9d2e-699e2578433d"
-      (reference "R8") (unit 1) (value "1K") (footprint "")
+      (reference "R8") (unit 1) (value "1K") (footprint "TestPoint:Two_Pad_Through_Hole_12.4mm")
     )
     (path "/81dcdae1-ae0e-4d8c-9bf2-1ad2e7737479"
-      (reference "R9") (unit 1) (value "1K") (footprint "")
+      (reference "R9") (unit 1) (value "1K") (footprint "TestPoint:Two_Pad_Through_Hole_12.4mm")
     )
     (path "/572a1812-167d-4df6-a541-c4a12c71e180"
-      (reference "R10") (unit 1) (value "1K") (footprint "")
+      (reference "R10") (unit 1) (value "1K") (footprint "TestPoint:Two_Pad_Through_Hole_12.4mm")
     )
     (path "/b3722303-ea62-4002-a830-59226134f53b"
-      (reference "R11") (unit 1) (value "1K") (footprint "")
+      (reference "R11") (unit 1) (value "1K") (footprint "TestPoint:Two_Pad_Through_Hole_12.4mm")
     )
     (path "/1a8342a5-15fc-454c-84eb-2b470c08f569/25dbed8c-d2ac-4070-9b7f-ca8dc63adfff"
@@
     )
     (path "/483eb092-6f48-48ea-b67d-8be254438fea"
-      (reference "Y3") (unit 1) (value "Crystal 3.58MHz") (footprint "")
-    )
-  )
+      (reference "Y3") (unit 1) (value "Crystal 3.58MHz") (footprint "TestPoint:Two_Pad_Through_Hole_10.4mm")
+    )
+  )
