File: SpaceCadet.kicad_sch (KiCad schematic)
At the start: 35 parts, among them J0 Conn_02x17_Odd_Even, J3_1 Conn_01x04, J3_2 Conn_01x04, U1 74LS154, U2 8048, Y3 Crystal 3.58MHz

Commit message: Modern EDA route, initial commit.
Parts:
- JP18, JP19, JP23, JP25, JP26, JP27, JP28, JP29, JP30, JP31, JP32: footprint (none) -> Jumper:SolderJumper-2_P1.3mm_Open_TrianglePad1.0x1.5mm
- JP20, JP21, JP22, JP24: footprint (none) -> Jumper:SolderJumper-2_P1.3mm_Bridged2Bar_Pad1.0x1.5mm
Connections:
- net COL0: no longer J3_1.1 (Pin_1)
- net COL1: no longer J3_1.2 (Pin_2)
- net COL2: now also JP31.1 (A); no longer J3_1.3 (Pin_3)
- net COL3: no longer J3_1.4 (Pin_4), JP31.1 (A)
- net COL4: no longer J3_2.1 (Pin_1)
- net COL5: no longer J3_2.2 (Pin_2)
- net COL6: no longer J3_2.3 (Pin_3)
- net COL7: no longer J3_2.4 (Pin_4)
- net ROW0: now also J3_1.1 (Pin_1)
- net ROW1: now also J3_1.2 (Pin_2)
- net ROW2: now also J3_1.3 (Pin_3)
- net ROW3: now also J3_1.4 (Pin_4)
- net ROW4: now also J3_2.1 (Pin_1)
- net ROW5: now also J3_2.2 (Pin_2); no longer JP25.1 (A)
- net ROW6: now also J3_2.3 (Pin_3)
- net ROW7: now also J3_2.4 (Pin_4), JP25.1 (A)
- net X2: now reaches C14.1, U2.3 (X2), Y3.1
- net X1: now reaches C13.1, U2.2 (X1), Y3.2

Commit message: Gerbers created.
Other:
- moved on the sheet: JP25
Changed lines of the file:
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@@
   (junction (at 53.34 80.645) (diameter 0) (color 0 0 0 0)
   )
-  (junction (at 178.435 107.95) (diameter 0) (color 0 0 0 0)
-  )
   (junction (at 120.65 107.95) (diameter 0) (color 0 0 0 0)
   )
@@
   )
   (junction (at 193.675 105.41) (diameter 0) (color 0 0 0 0)
+  )
+  (junction (at 178.435 105.41) (diameter 0) (color 0 0 0 0)
   )
   (junction (at 178.435 101.6) (diameter 0) (color 0 0 0 0)
@@
     (stroke (width 0) (type default) (color 0 0 0 0))
   )
+  (wire (pts (xy 178.435 105.41) (xy 178.435 110.49))
+    (stroke (width 0) (type default) (color 0 0 0 0))
+  )
   (wire (pts (xy 199.39 51.435) (xy 203.2 51.435))
     (stroke (width 0) (type default) (color 0 0 0 0))
@@
     (stroke (width 0) (type default) (color 0 0 0 0))
   )
-  (wire (pts (xy 175.895 107.95) (xy 178.435 107.95))
+  (wire (pts (xy 175.895 105.41) (xy 178.435 105.41))
     (stroke (width 0) (type default) (color 0 0 0 0))
   )
@@
     (stroke (width 0) (type default) (color 0 0 0 0))
   )
+  (wire (pts (xy 175.895 105.41) (xy 175.895 110.49))
+    (stroke (width 0) (type default) (color 0 0 0 0))
+  )
   (bus (pts (xy 183.515 133.985) (xy 183.515 135.255))
     (stroke (width 0) (type default) (color 0 0 0 0))
@@
     (stroke (width 0) (type default) (color 0 0 0 0))
   )
+  (wire (pts (xy 178.435 101.6) (xy 178.435 105.41))
+    (stroke (width 0) (type default) (color 0 0 0 0))
+  )
   (wire (pts (xy 199.39 40.005) (xy 203.2 40.005))
     (stroke (width 0) (type default) (color 0 0 0 0))
@@
     (stroke (width 0) (type default) (color 0 0 0 0))
   )
-  (wire (pts (xy 175.895 110.49) (xy 175.895 107.95))
-    (stroke (width 0) (type default) (color 0 0 0 0))
-  )
   (wire (pts (xy 66.675 42.545) (xy 74.93 42.545))
     (stroke (width 0) (type default) (color 0 0 0 0))
@@
     (stroke (width 0) (type default) (color 0 0 0 0))
   )
-  (wire (pts (xy 178.435 107.95) (xy 178.435 110.49))
-    (stroke (width 0) (type default) (color 0 0 0 0))
-  )
   (bus (pts (xy 59.055 137.16) (xy 59.055 134.62))
     (stroke (width 0) (type default) (color 0 0 0 0))
@@
   )
   (polyline (pts (xy 228.6 19.685) (xy 228.6 115.57))
-    (stroke (width 0) (type default) (color 0 0 0 0))
-  )
-  (wire (pts (xy 178.435 101.6) (xy 178.435 107.95))
     (stroke (width 0) (type default) (color 0 0 0 0))
   )
@@
     (effects (font (size 1.27 1.27)) (justify left bottom))
   )
+  (label "GND" (at 188.595 110.49 90)
+    (effects (font (size 1.27 1.27)) (justify left bottom))
+  )
   (label "COL7" (at 95.25 152.4 0) (fields_autoplaced)
     (effects (font (size 1.27 1.27)) (justify left bottom))
@@
   )
   (label "ROW1" (at 68.58 65.405 0) (fields_autoplaced)
+    (effects (font (size 1.27 1.27)) (justify left bottom))
+  )
+  (label "+5V" (at 178.435 110.49 90)
     (effects (font (size 1.27 1.27)) (justify left bottom))
   )
@@
   (symbol (lib_id "Jumper:Jumper_2_Bridged") (at 208.28 62.865 0) (unit 1)
     (in_bom yes) (on_board yes)
-    (property "Reference" "JP24" (id 0) (at 208.28 61.595 0))
+    (property "Reference" "JP24" (id 0) (at 208.28 64.77 0))
     (property "Value" "Jumper Bridged" (id 1) (at 191.135 62.865 0)
       (effects (font (size 1.27 1.27)) (justify right))
@@
   (symbol (lib_id "Jumper:Jumper_2_Open") (at 260.35 92.71 0) (unit 1)
     (in_bom yes) (on_board yes)
-    (property "Reference" "JP29" (id 0) (at 262.255 93.98 0)
-      (effects (font (size 1.27 1.27)) (justify right))
-    )
+    (property "Reference" "JP29" (id 0) (at 260.35 94.615 0))
     (property "Value" "Jumper Open" (id 1) (at 243.205 92.71 0)
       (effects (font (size 1.27 1.27)) (justify right))
@@
   (symbol (lib_id "Jumper:Jumper_2_Bridged") (at 208.28 40.005 0) (unit 1)
     (in_bom yes) (on_board yes)
-    (property "Reference" "JP20" (id 0) (at 208.28 38.735 0))
+    (property "Reference" "JP20" (id 0) (at 208.28 41.91 0))
     (property "Value" "Jumper Bridged" (id 1) (at 191.135 40.005 0)
       (effects (font (size 1.27 1.27)) (justify right))
@@
   (symbol (lib_id "Jumper:Jumper_2_Open") (at 260.35 104.14 0) (unit 1)
     (in_bom yes) (on_board yes)
-    (property "Reference" "JP31" (id 0) (at 262.255 105.41 0)
-      (effects (font (size 1.27 1.27)) (justify right))
-    )
+    (property "Reference" "JP31" (id 0) (at 260.35 106.045 0))
     (property "Value" "Jumper Open" (id 1) (at 243.205 104.14 0)
       (effects (font (size 1.27 1.27)) (justify right))
@@
   (symbol (lib_id "Jumper:Jumper_2_Open") (at 260.35 109.855 0) (unit 1)
     (in_bom yes) (on_board yes)
-    (property "Reference" "JP32" (id 0) (at 262.255 111.125 0)
-      (effects (font (size 1.27 1.27)) (justify right))
-    )
+    (property "Reference" "JP32" (id 0) (at 260.35 111.76 0))
     (property "Value" "Jumper Open" (id 1) (at 243.205 109.855 0)
       (effects (font (size 1.27 1.27)) (justify right))
@@
   (symbol (lib_id "Jumper:Jumper_2_Open") (at 260.35 98.425 0) (unit 1)
     (in_bom yes) (on_board yes)
-    (property "Reference" "JP30" (id 0) (at 262.255 99.695 0)
-      (effects (font (size 1.27 1.27)) (justify right))
-    )
+    (property "Reference" "JP30" (id 0) (at 260.35 100.33 0))
     (property "Value" "Jumper Open" (id 1) (at 243.205 98.425 0)
       (effects (font (size 1.27 1.27)) (justify right))
@@
   (symbol (lib_id "Jumper:Jumper_2_Open") (at 260.35 75.565 0) (unit 1)
     (in_bom yes) (on_board yes)
-    (property "Reference" "JP26" (id 0) (at 262.255 76.835 0)
-      (effects (font (size 1.27 1.27)) (justify right))
-    )
+    (property "Reference" "JP26" (id 0) (at 260.35 77.47 0))
     (property "Value" "Jumper Open" (id 1) (at 243.205 75.565 0)
       (effects (font (size 1.27 1.27)) (justify right))
@@
     (pin "2")
   )
-  (symbol (lib_id "Jumper:Jumper_2_Open") (at 260.35 69.85 0) (mirror x) (unit 1)
-    (in_bom yes) (on_board yes)
-    (property "Reference" "JP25" (id 0) (at 262.89 67.945 0)
-      (effects (font (size 1.27 1.27)) (justify right))
-    )
+  (symbol (lib_id "Jumper:Jumper_2_Open") (at 260.35 69.85 0) (unit 1)
+    (in_bom yes) (on_board yes)
+    (property "Reference" "JP25" (id 0) (at 260.35 71.755 0))
     (property "Value" "Jumper Open" (id 1) (at 243.205 69.85 0)
       (effects (font (size 1.27 1.27)) (justify right))
@@
   (symbol (lib_id "Jumper:Jumper_2_Open") (at 260.35 34.29 0) (unit 1)
     (in_bom yes) (on_board yes)
-    (property "Reference" "JP19" (id 0) (at 262.255 31.75 0)
-      (effects (font (size 1.27 1.27)) (justify right))
-    )
+    (property "Reference" "JP19" (id 0) (at 260.35 36.195 0))
     (property "Value" "Jumper Open" (id 1) (at 243.205 34.29 0)
       (effects (font (size 1.27 1.27)) (justify right))
@@
   (symbol (lib_id "Jumper:Jumper_2_Open") (at 260.35 28.575 0) (unit 1)
     (in_bom yes) (on_board yes)
-    (property "Reference" "JP18" (id 0) (at 262.255 26.035 0)
-      (effects (font (size 1.27 1.27)) (justify right))
-    )
+    (property "Reference" "JP18" (id 0) (at 260.35 30.48 0))
     (property "Value" "Jumper Open" (id 1) (at 243.205 28.575 0)
       (effects (font (size 1.27 1.27)) (justify right))
@@
   (symbol (lib_id "Jumper:Jumper_2_Open") (at 260.35 57.15 0) (unit 1)
     (in_bom yes) (on_board yes)
-    (property "Reference" "JP23" (id 0) (at 262.255 54.61 0)
-      (effects (font (size 1.27 1.27)) (justify right))
-    )
+    (property "Reference" "JP23" (id 0) (at 260.35 59.055 0))
     (property "Value" "Jumper Open" (id 1) (at 243.205 57.15 0)
       (effects (font (size 1.27 1.27)) (justify right))
@@
   (symbol (lib_id "Jumper:Jumper_2_Bridged") (at 208.28 45.72 0) (unit 1)
     (in_bom yes) (on_board yes)
-    (property "Reference" "JP21" (id 0) (at 208.28 44.45 0))
+    (property "Reference" "JP21" (id 0) (at 208.28 47.625 0))
     (property "Value" "Jumper Bridged" (id 1) (at 191.135 45.72 0)
       (effects (font (size 1.27 1.27)) (justify right))
@@
   (symbol (lib_id "Jumper:Jumper_2_Open") (at 260.35 86.995 0) (unit 1)
     (in_bom yes) (on_board yes)
-    (property "Reference" "JP28" (id 0) (at 262.255 88.265 0)
-      (effects (font (size 1.27 1.27)) (justify right))
-    )
+    (property "Reference" "JP28" (id 0) (at 260.35 88.9 0))
     (property "Value" "Jumper Open" (id 1) (at 243.205 86.995 0)
       (effects (font (size 1.27 1.27)) (justify right))
@@
   (symbol (lib_id "Jumper:Jumper_2_Bridged") (at 208.28 51.435 0) (unit 1)
     (in_bom yes) (on_board yes)
-    (property "Reference" "JP22" (id 0) (at 208.28 50.165 0))
+    (property "Reference" "JP22" (id 0) (at 208.28 53.34 0))
     (property "Value" "Jumper Bridged" (id 1) (at 191.135 51.435 0)
       (effects (font (size 1.27 1.27)) (justify right))
@@
   (symbol (lib_id "Jumper:Jumper_2_Open") (at 260.35 81.28 0) (unit 1)
     (in_bom yes) (on_board yes)
-    (property "Reference" "JP27" (id 0) (at 262.255 82.55 0)
-      (effects (font (size 1.27 1.27)) (justify right))
-    )
+    (property "Reference" "JP27" (id 0) (at 260.35 83.185 0))
     (property "Value" "Jumper Open" (id 1) (at 243.205 81.28 0)
       (effects (font (size 1.27 1.27)) (justify right))
@@
       (reference "#PWR0113") (unit 1) (value "+5V") (footprint "")
     )
+    (path "/1a8342a5-15fc-454c-84eb-2b470c08f569/44de499e-d74e-4a0b-ad44-b5559c965905"
+      (reference "#PWR?") (unit 1) (value "+5V") (footprint "")
+    )
     (path "/4b693529-fe06-44af-a160-67a5ffd8665d"

Commit message: Updated the rounded variant.
Parts:
- C12, C13, C14, Y3: footprint (none) -> TestPoint:Two_Pad_Through_Hole_10.4mm
- C15: footprint (none) -> TestPoint:Two_Pad_Through_Hole_10.4mm; PossibleFootprint Capacitor_THT:C_Axial_L3.8mm_D2.6mm_P12.50mm_Horizontal -> (none)
- C16: footprint (none) -> TestPoint:Two_Pad_Through_Hole_20mm; PossibleFootprint Capacitor_THT:CP_Axial_L25.0mm_D10.0mm_P30.00mm_Horizontal -> (none)
- C17: footprint (none) -> TestPoint:Two_Pad_Through_Hole_12mm
- R10, R11, R4, R5, R6, R7, R8, R9: footprint (none) -> TestPoint:Two_Pad_Through_Hole_12.4mm
Changed lines of the file:
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@@
     (property "Reference" "C16" (id 0) (at 181.61 95.25 90))
     (property "Value" "22uF 15v" (id 1) (at 191.135 95.25 90))
-    (property "Footprint" "" (id 2) (at 184.785 96.52 0)
+    (property "Footprint" "TestPoint:Two_Pad_Through_Hole_20mm" (id 2) (at 184.785 96.52 0)
       (effects (font (size 1.27 1.27)) hide)
     )
@@
       (effects (font (size 1.27 1.27)) hide)
     )
-    (property "PossibleFootprint" "Capacitor_THT:CP_Axial_L25.0mm_D10.0mm_P30.00mm_Horizontal" (id 4) (at 184.785 96.52 90)
+    (property "PossibleFootprint" "" (id 4) (at 184.785 96.52 90)
       (effects (font (size 1.27 1.27)) hide)
     )
@@
     (property "Reference" "Y3" (id 0) (at 120.65 93.0275 0))
     (property "Value" "Crystal 3.58MHz" (id 1) (at 120.65 94.7897 0))
-    (property "Footprint" "" (id 2) (at 120.65 98.425 0)
+    (property "Footprint" "TestPoint:Two_Pad_Through_Hole_10.4mm" (id 2) (at 120.65 98.425 0)
       (effects (font (size 1.27 1.27)) hide)
     )
@@
     (property "Reference" "C12" (id 0) (at 88.9 120.015 90))
     (property "Value" "10pF" (id 1) (at 89.535 121.92 90))
-    (property "Footprint" "" (id 2) (at 89.535 122.2248 0)
+    (property "Footprint" "TestPoint:Two_Pad_Through_Hole_10.4mm" (id 2) (at 89.535 122.2248 0)
       (effects (font (size 1.27 1.27)) hide)
     )
@@
     (property "Reference" "C15" (id 0) (at 182.88 100.33 90))
     (property "Value" "15pF" (id 1) (at 182.245 102.87 90))
-    (property "Footprint" "" (id 2) (at 185.42 101.6 0)
+    (property "Footprint" "TestPoint:Two_Pad_Through_Hole_10.4mm" (id 2) (at 185.42 101.6 0)
       (effects (font (size 1.27 1.27)) hide)
     )
@@
       (effects (font (size 1.27 1.27)) hide)
     )
-    (property "PossibleFootprint" "Capacitor_THT:C_Axial_L3.8mm_D2.6mm_P12.50mm_Horizontal" (id 4) (at 185.42 101.6 90)
+    (property "PossibleFootprint" "" (id 4) (at 182.245 80.645 90)
       (effects (font (size 1.27 1.27)) hide)
     )
@@
     (property "Reference" "R4" (id 0) (at 50.8 95.25 90))
     (property "Value" "1K" (id 1) (at 50.165 86.36 90))
-    (property "Footprint" "" (id 2) (at 49.784 89.281 90)
+    (property "Footprint" "TestPoint:Two_Pad_Through_Hole_12.4mm" (id 2) (at 49.784 89.281 90)
       (effects (font (size 1.27 1.27)) hide)
     )
@@
     (property "Reference" "R10" (id 0) (at 38.1 95.25 90))
     (property "Value" "1K" (id 1) (at 37.465 86.36 90))
-    (property "Footprint" "" (id 2) (at 37.084 89.281 90)
+    (property "Footprint" "TestPoint:Two_Pad_Through_Hole_12.4mm" (id 2) (at 37.084 89.281 90)
       (effects (font (size 1.27 1.27)) hide)
     )
@@
     (property "Reference" "R6" (id 0) (at 48.26 95.25 90))
     (property "Value" "1K" (id 1) (at 47.625 86.36 90))
-    (property "Footprint" "" (id 2) (at 47.244 89.281 90)
+    (property "Footprint" "TestPoint:Two_Pad_Through_Hole_12.4mm" (id 2) (at 47.244 89.281 90)
       (effects (font (size 1.27 1.27)) hide)
     )
@@
     (property "Reference" "R5" (id 0) (at 53.34 95.25 90))
     (property "Value" "1K" (id 1) (at 52.705 86.36 90))
-    (property "Footprint" "" (id 2) (at 52.324 89.281 90)
+    (property "Footprint" "TestPoint:Two_Pad_Through_Hole_12.4mm" (id 2) (at 52.324 89.281 90)
       (effects (font (size 1.27 1.27)) hide)
     )
@@
     (property "Reference" "R9" (id 0) (at 40.64 95.25 90))
     (property "Value" "1K" (id 1) (at 40.005 86.36 90))
-    (property "Footprint" "" (id 2) (at 39.624 89.281 90)
+    (property "Footprint" "TestPoint:Two_Pad_Through_Hole_12.4mm" (id 2) (at 39.624 89.281 90)
       (effects (font (size 1.27 1.27)) hide)
     )
@@
       (effects (font (size 1.27 1.27)) (justify left))
     )
-    (property "Footprint" "" (id 2) (at 115.9002 107.95 0)
+    (property "Footprint" "TestPoint:Two_Pad_Through_Hole_10.4mm" (id 2) (at 115.9002 107.95 0)
       (effects (font (size 1.27 1.27)) hide)
     )
@@
       (effects (font (size 1.27 1.27)) (justify left))
     )
-    (property "Footprint" "" (id 2) (at 127.3302 107.95 0)
+    (property "Footprint" "TestPoint:Two_Pad_Through_Hole_10.4mm" (id 2) (at 127.3302 107.95 0)
       (effects (font (size 1.27 1.27)) hide)
     )
@@
     (property "Reference" "C17" (id 0) (at 203.2 131.445 90))
     (property "Value" "4.7uF 25v" (id 1) (at 200.66 133.35 90))
-    (property "Footprint" "" (id 2) (at 199.39 130.175 0)
+    (property "Footprint" "TestPoint:Two_Pad_Through_Hole_12mm" (id 2) (at 199.39 130.175 0)
       (effects (font (size 1.27 1.27)) hide)
     )
@@
     (property "Reference" "R7" (id 0) (at 45.72 95.25 90))
     (property "Value" "1K" (id 1) (at 45.085 86.36 90))
-    (property "Footprint" "" (id 2) (at 44.704 89.281 90)
+    (property "Footprint" "TestPoint:Two_Pad_Through_Hole_12.4mm" (id 2) (at 44.704 89.281 90)
       (effects (font (size 1.27 1.27)) hide)
     )
@@
     (property "Reference" "R11" (id 0) (at 35.56 95.25 90))
     (property "Value" "1K" (id 1) (at 34.925 86.36 90))
-    (property "Footprint" "" (id 2) (at 34.544 89.281 90)
+    (property "Footprint" "TestPoint:Two_Pad_Through_Hole_12.4mm" (id 2) (at 34.544 89.281 90)
       (effects (font (size 1.27 1.27)) hide)
     )
@@
     (property "Reference" "R8" (id 0) (at 43.18 95.25 90))
     (property "Value" "1K" (id 1) (at 42.545 86.36 90))
-    (property "Footprint" "" (id 2) (at 42.164 89.281 90)
+    (property "Footprint" "TestPoint:Two_Pad_Through_Hole_12.4mm" (id 2) (at 42.164 89.281 90)
       (effects (font (size 1.27 1.27)) hide)
     )
@@
     )
     (path "/1a8342a5-15fc-454c-84eb-2b470c08f569/44de499e-d74e-4a0b-ad44-b5559c965905"
-      (reference "#PWR?") (unit 1) (value "+5V") (footprint "")
+      (reference "#PWR0114") (unit 1) (value "+5V") (footprint "")
     )
     (path "/4b693529-fe06-44af-a160-67a5ffd8665d"
-      (reference "C12") (unit 1) (value "10pF") (footprint "")
+      (reference "C12") (unit 1) (value "10pF") (footprint "TestPoint:Two_Pad_Through_Hole_10.4mm")
     )
     (path "/8cff2a90-9996-4fb8-b834-7ba83869fd3b"
-      (reference "C13") (unit 1) (value "10pF") (footprint "")
+      (reference "C13") (unit 1) (value "10pF") (footprint "TestPoint:Two_Pad_Through_Hole_10.4mm")
     )
     (path "/8579f6ff-d916-43cb-9f3a-9ef7b7dec6ac"
-      (reference "C14") (unit 1) (value "10pF") (footprint "")
+      (reference "C14") (unit 1) (value "10pF") (footprint "TestPoint:Two_Pad_Through_Hole_10.4mm")
     )
     (path "/4ec161d3-1c9b-4ea4-8ce3-cad9856a00a1"
-      (reference "C15") (unit 1) (value "15pF") (footprint "")
+      (reference "C15") (unit 1) (value "15pF") (footprint "TestPoint:Two_Pad_Through_Hole_10.4mm")
     )
     (path "/0483c138-e6fc-4834-bde0-ce6afaa0b50e"
-      (reference "C16") (unit 1) (value "22uF 15v") (footprint "")
+      (reference "C16") (unit 1) (value "22uF 15v") (footprint "TestPoint:Two_Pad_Through_Hole_20mm")
     )
     (path "/94b91b8a-0258-4cda-a957-e6f302c9f04e"
-      (reference "C17") (unit 1) (value "4.7uF 25v") (footprint "")
+      (reference "C17") (unit 1) (value "4.7uF 25v") (footprint "TestPoint:Two_Pad_Through_Hole_12mm")
     )
     (path "/1ea855f8-a5b1-424e-a642-dd01e460d8f4"
@@
     )
     (path "/4ed57943-0461-493e-8f46-26d1eea10a82"
-      (reference "R4") (unit 1) (value "1K") (footprint "")
+      (reference "R4") (unit 1) (value "1K") (footprint "TestPoint:Two_Pad_Through_Hole_12.4mm")
     )
     (path "/7ef65beb-8399-4097-ac13-2d05b63259d4"
-      (reference "R5") (unit 1) (value "1K") (footprint "")
+      (reference "R5") (unit 1) (value "1K") (footprint "TestPoint:Two_Pad_Through_Hole_12.4mm")
     )
     (path "/585e9c7f-d46a-4180-8342-4d9663c8f2cc"
-      (reference "R6") (unit 1) (value "1K") (footprint "")
+      (reference "R6") (unit 1) (value "1K") (footprint "TestPoint:Two_Pad_Through_Hole_12.4mm")
     )
     (path "/b1af4875-6c7a-4214-901c-5aeac72b67c9"
-      (reference "R7") (unit 1) (value "1K") (footprint "")
+      (reference "R7") (unit 1) (value "1K") (footprint "TestPoint:Two_Pad_Through_Hole_12.4mm")
     )
     (path "/e80dacb6-6a6c-44ed-9d2e-699e2578433d"
-      (reference "R8") (unit 1) (value "1K") (footprint "")
+      (reference "R8") (unit 1) (value "1K") (footprint "TestPoint:Two_Pad_Through_Hole_12.4mm")
     )
     (path "/81dcdae1-ae0e-4d8c-9bf2-1ad2e7737479"
-      (reference "R9") (unit 1) (value "1K") (footprint "")
+      (reference "R9") (unit 1) (value "1K") (footprint "TestPoint:Two_Pad_Through_Hole_12.4mm")
     )
     (path "/572a1812-167d-4df6-a541-c4a12c71e180"
-      (reference "R10") (unit 1) (value "1K") (footprint "")
+      (reference "R10") (unit 1) (value "1K") (footprint "TestPoint:Two_Pad_Through_Hole_12.4mm")
     )
     (path "/b3722303-ea62-4002-a830-59226134f53b"
-      (reference "R11") (unit 1) (value "1K") (footprint "")
+      (reference "R11") (unit 1) (value "1K") (footprint "TestPoint:Two_Pad_Through_Hole_12.4mm")
     )
     (path "/1a8342a5-15fc-454c-84eb-2b470c08f569/25dbed8c-d2ac-4070-9b7f-ca8dc63adfff"
@@
     )
     (path "/483eb092-6f48-48ea-b67d-8be254438fea"
-      (reference "Y3") (unit 1) (value "Crystal 3.58MHz") (footprint "")
-    )
-  )
+      (reference "Y3") (unit 1) (value "Crystal 3.58MHz") (footprint "TestPoint:Two_Pad_Through_Hole_10.4mm")
+    )
+  )
