File: SpaceCadet-rounded.kicad_pcb (KiCad board)
At the start: 2 copper layers, 469 x 166.6 mm, 217 parts, among them J0 Conn_02x17_Odd_Even, J3_1 Conn_01x04, J3_2 Conn_01x04, SW1 SD_4B3E, SW10 SD_4B3E, SW100 SD_4B3E, SW101 SD_4B3E, SW102 SD_4B3E, SW103 SD_4B3E, SW104 SD_4B3E, SW105 SD_4B3E, SW106 SD_4B3E, SW107 SD_4B3E, SW108 SD_4B3E, SW109 SD_4B3E, SW11 SD_4B3E, SW110 SD_4B3E, SW111 SD_4B3E, SW112 SD_4B3E, SW113 SD_4B3E, SW114 SD_4B3E, SW115 SD_4B3E, SW116 SD_4B3E, SW117 SD_4B3E, SW118 SD_4B3E, SW119 SD_4B3E, SW12 SD_4B3E, SW120 SD_4B3E, SW121 SD_4B3E, SW122 SD_4B3E, SW122a0 SD_4B3E, SW123 SD_4B3E, SW123a0 SD_4B3E, SW124 SD_4B3E, SW124a0 SD_4B3E, SW125 SD_4B3E, SW126 SD_4B3E, SW127 SD_4B3E, SW128 SD_4B3E, SW13 SD_4B3E, SW14 SD_4B3E, SW15 SD_4B3E, SW16 SD_4B3E, SW17 SD_4B3E, SW18 SD_4B3E, SW19 SD_4B3E, SW2 SD_4B3E, SW20 SD_4B3E, SW21 SD_4B3E, SW22 SD_4B3E, SW23 SD_4B3E, SW24 SD_4B3E, SW25 SD_4B3E, SW26 SD_4B3E, SW27 SD_4B3E, SW28 SD_4B3E, SW29 SD_4B3E, SW3 SD_4B3E, SW30 SD_4B3E, SW31 SD_4B3E, SW32 SD_4B3E, SW33 SD_4B3E, SW34 SD_4B3E, SW35 SD_4B3E, SW36 SD_4B3E, SW37 SD_4B3E, SW38 SD_4B3E, SW39 SD_4B3E, SW4 SD_4B3E, SW40 SD_4B3E, SW41 SD_4B3E, SW42 SD_4B3E, SW43 SD_4B3E, SW44 SD_4B3E, SW45 SD_4B3E, SW46 SD_4B3E, SW47 SD_4B3E, SW48 SD_4B3E, SW49 SD_4B3E, SW5 SD_4B3E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

Commit message: Updated the rounded variant.
Parts:
- removed ? (x28): , 
- removed the REF** at (340.6, 108.5)
- removed the REF** at (340.6, 96.0)
- added C12: 10pF, TestPoint:Two_Pad_Through_Hole_10.4mm, F.Cu at (230.7, 104.9)
- added C13: 10pF, TestPoint:Two_Pad_Through_Hole_10.4mm, F.Cu at (301.6, 114.8)
- added C14: 10pF, TestPoint:Two_Pad_Through_Hole_10.4mm, F.Cu at (301.6, 117.9)
- added C15: 15pF, TestPoint:Two_Pad_Through_Hole_10.4mm, F.Cu at (524.6, 111.2)
- added C16: 22uF 15v, TestPoint:Two_Pad_Through_Hole_20mm, F.Cu at (515.7, 117.0)
- added C17: 4.7uF 25v, TestPoint:Two_Pad_Through_Hole_12mm, F.Cu at (509.8, 111.6)
- added R10: 1K, TestPoint:Two_Pad_Through_Hole_12.4mm, F.Cu at (422.0, 92.4)
- added R11: 1K, TestPoint:Two_Pad_Through_Hole_12.4mm, F.Cu at (419.5, 89.8)
- added R4: 1K, TestPoint:Two_Pad_Through_Hole_12.4mm, F.Cu at (340.6, 102.2)
- added R5: 1K, TestPoint:Two_Pad_Through_Hole_12.4mm, F.Cu at (343.9, 102.2)
- added R6: 1K, TestPoint:Two_Pad_Through_Hole_12.4mm, F.Cu at (383.8, 98.0)
- added R7: 1K, TestPoint:Two_Pad_Through_Hole_12.4mm, F.Cu at (389.0, 95.8)
- added R8: 1K, TestPoint:Two_Pad_Through_Hole_12.4mm, F.Cu at (402.4, 98.0)
- added R9: 1K, TestPoint:Two_Pad_Through_Hole_12.4mm, F.Cu at (419.5, 94.9)
- added Y3: Crystal 3.58MHz, TestPoint:Two_Pad_Through_Hole_10.4mm, F.Cu at (301.8, 111.5)
Connections:
- U1 pad 10: COL9 -> /COL9
- U1 pad 11: COL10 -> /COL10
- U1 pad 13: COL11 -> /COL11
- U1 pad 14: COL12 -> /COL12
- U1 pad 15: COL13 -> /COL13
- U1 pad 16: COL14 -> /COL14
- U1 pad 17: COL15 -> /COL15
- U1 pad 4: COL3 -> /COL3
- U1 pad 6: COL5 -> /COL5
- U1 pad 7: COL6 -> /COL6
- U1 pad 8: COL7 -> /COL7
- U1 pad 9: COL8 -> /COL8
Routing:
- net GND: track 962.5 -> 1015.2 mm
- net COL11: track 362.4 -> 350.6 mm
- net COL5: track 866.6 -> 855.3 mm
- net COL12: track 354.6 -> 343.3 mm
- net COL9: track 428.2 -> 417.5 mm
- net COL13: track 506.4 -> 495.8 mm
- net COL7: track 718.1 -> 708.7 mm
- net COL10: track 378.6 -> 369.5 mm
- net COL15: track 531.6 -> 522.6 mm
- net COL14: track 305.0 -> 296.6 mm
- net COL8: track 480.0 -> 472.6 mm
- net COL4: track 803.8 -> 796.8 mm
- net +5V: track 3677.7 -> 3673.8 mm
- net ROW6: track 542.1 -> 538.2 mm
- net COL2: track 951.5 -> 948.0 mm
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Other:
- board text added: "Trace extends to the edge of the board. -->"
