File: SpaceCadet.kicad_pcb (KiCad board)
At the start: 2 copper layers, 469 x 166.6 mm, 202 parts, among them J0 Conn_02x17_Odd_Even, J3_1 Conn_01x04, J3_2 Conn_01x04, SW1 SD_4B3E, SW10 SD_4B3E, SW100 SD_4B3E, SW101 SD_4B3E, SW102 SD_4B3E, SW103 SD_4B3E, SW104 SD_4B3E, SW105 SD_4B3E, SW106 SD_4B3E, SW107 SD_4B3E, SW108 SD_4B3E, SW109 SD_4B3E, SW11 SD_4B3E, SW110 SD_4B3E, SW111 SD_4B3E, SW112 SD_4B3E, SW113 SD_4B3E, SW114 SD_4B3E, SW115 SD_4B3E, SW116 SD_4B3E, SW117 SD_4B3E, SW118 SD_4B3E, SW119 SD_4B3E, SW12 SD_4B3E, SW120 SD_4B3E, SW121 SD_4B3E, SW122 SD_4B3E, SW122a0 SD_4B3E, SW123 SD_4B3E, SW123a0 SD_4B3E, SW124 SD_4B3E, SW124a0 SD_4B3E, SW125 SD_4B3E, SW126 SD_4B3E, SW127 SD_4B3E, SW128 SD_4B3E, SW13 SD_4B3E, SW14 SD_4B3E, SW15 SD_4B3E, SW16 SD_4B3E, SW17 SD_4B3E, SW18 SD_4B3E, SW19 SD_4B3E, SW2 SD_4B3E, SW20 SD_4B3E, SW21 SD_4B3E, SW22 SD_4B3E, SW23 SD_4B3E, SW24 SD_4B3E, SW25 SD_4B3E, SW26 SD_4B3E, SW27 SD_4B3E, SW28 SD_4B3E, SW29 SD_4B3E, SW3 SD_4B3E, SW30 SD_4B3E, SW31 SD_4B3E, SW32 SD_4B3E, SW33 SD_4B3E, SW34 SD_4B3E, SW35 SD_4B3E, SW36 SD_4B3E, SW37 SD_4B3E, SW38 SD_4B3E, SW39 SD_4B3E, SW4 SD_4B3E, SW40 SD_4B3E, SW41 SD_4B3E, SW42 SD_4B3E, SW43 SD_4B3E, SW44 SD_4B3E, SW45 SD_4B3E, SW46 SD_4B3E, SW47 SD_4B3E, SW48 SD_4B3E, SW49 SD_4B3E, SW5 SD_4B3E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

Commit message: Modern EDA route, initial commit.
Parts:
- added JP18: Jumper Open, Jumper:SolderJumper-2_P1.3mm_Open_TrianglePad1.0x1.5mm, F.Cu at (347.9, 111.3)
- added JP19: Jumper Open, Jumper:SolderJumper-2_P1.3mm_Open_TrianglePad1.0x1.5mm, F.Cu at (368.1, 120.4)
- added JP20: Jumper Bridged, Jumper:SolderJumper-2_P1.3mm_Bridged2Bar_Pad1.0x1.5mm, F.Cu at (446.0, 110.8)
- added JP21: Jumper Bridged, Jumper:SolderJumper-2_P1.3mm_Bridged2Bar_Pad1.0x1.5mm, F.Cu at (446.0, 107.2)
- added JP22: Jumper Bridged, Jumper:SolderJumper-2_P1.3mm_Bridged2Bar_Pad1.0x1.5mm, F.Cu at (446.0, 103.7)
- added JP23: Jumper Open, Jumper:SolderJumper-2_P1.3mm_Open_TrianglePad1.0x1.5mm, F.Cu at (473.9, 124.6)
- added JP24: Jumper Bridged, Jumper:SolderJumper-2_P1.3mm_Bridged2Bar_Pad1.0x1.5mm, F.Cu at (478.3, 121.2)
- added JP25: Jumper Open, Jumper:SolderJumper-2_P1.3mm_Open_TrianglePad1.0x1.5mm, F.Cu at (75.7, 95.1)
- added JP26: Jumper Open, Jumper:SolderJumper-2_P1.3mm_Open_TrianglePad1.0x1.5mm, F.Cu at (82.0, 95.1)
- added JP27: Jumper Open, Jumper:SolderJumper-2_P1.3mm_Open_TrianglePad1.0x1.5mm, F.Cu at (95.1, 97.6)
- added JP28: Jumper Open, Jumper:SolderJumper-2_P1.3mm_Open_TrianglePad1.0x1.5mm, F.Cu at (98.2, 97.6)
- added JP29: Jumper Open, Jumper:SolderJumper-2_P1.3mm_Open_TrianglePad1.0x1.5mm, F.Cu at (112.6, 97.6)
- added JP30: Jumper Open, Jumper:SolderJumper-2_P1.3mm_Open_TrianglePad1.0x1.5mm, F.Cu at (119.9, 97.6)
- added JP31: Jumper Open, Jumper:SolderJumper-2_P1.3mm_Open_TrianglePad1.0x1.5mm, F.Cu at (125.2, 97.6)
- added JP32: Jumper Open, Jumper:SolderJumper-2_P1.3mm_Open_TrianglePad1.0x1.5mm, F.Cu at (134.7, 97.6)
- moved ? 6.12 mm to (503.8, 111.5)
- moved ? 4.81 mm to (505.8, 117.1)
- moved ? 0.57 mm to (516.0, 111.5)
Connections:
- ? pad 1: (no net) -> +5V (x3)
- ? pad 1: (no net) -> RESET
- ? pad 1: (no net) -> ROW4
- ? pad 1: (no net) -> GND (x12)
- ? pad 1: (no net) -> ROW2
- ? pad 1: (no net) -> ROW1
- ? pad 1: (no net) -> /X1 (x2)
- ? pad 1: (no net) -> /X2 (x2)
- ? pad 1: (no net) -> ROW7
- ? pad 1: (no net) -> ROW0
- ? pad 1: (no net) -> ROW5
- ? pad 1: (no net) -> ROW3
- J3_1 pad 1: COL0 -> ROW0
- J3_1 pad 2: COL1 -> ROW1
- J3_1 pad 3: COL2 -> ROW2
- J3_1 pad 4: COL3 -> ROW3
- J3_2 pad 1: COL4 -> ROW4
- J3_2 pad 2: COL5 -> ROW5
- J3_2 pad 3: COL6 -> ROW6
- J3_2 pad 4: COL7 -> ROW7
- REF** pad 1: (no net) -> ROW6
- SW1 pad 2: GND -> +5V
- SW10 pad 2: GND -> +5V
- SW100 pad 2: GND -> +5V
- SW101 pad 2: GND -> +5V
- SW102 pad 2: GND -> +5V
- SW103 pad 2: GND -> +5V
- SW104 pad 2: GND -> +5V
- SW105 pad 2: GND -> +5V
- SW106 pad 2: GND -> +5V
- SW107 pad 2: GND -> +5V
- SW108 pad 2: GND -> +5V
- SW109 pad 2: GND -> +5V
- SW11 pad 2: GND -> +5V
- SW110 pad 2: GND -> +5V
- SW111 pad 2: GND -> +5V
- SW112 pad 2: GND -> +5V
- SW113 pad 2: GND -> +5V
- SW114 pad 2: GND -> +5V
- SW115 pad 2: GND -> +5V
- SW116 pad 2: GND -> +5V
- SW117 pad 2: GND -> +5V
- SW118 pad 2: GND -> +5V
- SW119 pad 2: GND -> +5V
- SW119 pad 3: COL0 -> COL1
- SW12 pad 2: GND -> +5V
- SW120 pad 2: GND -> +5V
- SW120 pad 3: COL1 -> COL0
- SW121 pad 2: GND -> +5V
- SW122 pad 2: GND -> +5V
- SW122a0 pad 2: GND -> +5V
- SW123 pad 2: GND -> +5V
- SW123a0 pad 2: GND -> +5V
- SW124 pad 2: GND -> +5V
- SW124a0 pad 2: GND -> +5V
- SW125 pad 2: GND -> +5V
- SW126 pad 2: GND -> +5V
- SW127 pad 2: GND -> +5V
- SW128 pad 2: GND -> +5V
- SW13 pad 2: GND -> +5V
- SW14 pad 2: GND -> +5V
- SW15 pad 2: GND -> +5V
- SW16 pad 2: GND -> +5V
- SW17 pad 2: GND -> +5V
- SW18 pad 2: GND -> +5V
- SW19 pad 2: GND -> +5V
- SW2 pad 2: GND -> +5V
- SW2 pad 3: unconnected-(SW2-Pad3) -> COL1
- SW20 pad 2: GND -> +5V
- SW21 pad 2: GND -> +5V
- SW22 pad 2: GND -> +5V
- SW22 pad 3: COL1 -> COL0
- SW23 pad 2: GND -> +5V
- SW23 pad 3: COL0 -> COL1
- SW24 pad 2: GND -> +5V
- SW25 pad 2: GND -> +5V
- SW26 pad 2: GND -> +5V
- SW27 pad 2: GND -> +5V
- SW28 pad 2: GND -> +5V
- SW29 pad 2: GND -> +5V
- SW3 pad 2: GND -> +5V
- SW3 pad 3: unconnected-(SW3-Pad3) -> COL0
- SW30 pad 2: GND -> +5V
- SW31 pad 2: GND -> +5V
- SW32 pad 2: GND -> +5V
- SW33 pad 2: GND -> +5V
- SW34 pad 2: GND -> +5V
- SW35 pad 2: GND -> +5V
- SW36 pad 2: GND -> +5V
- SW37 pad 2: GND -> +5V
- SW38 pad 2: GND -> +5V
- SW39 pad 2: GND -> +5V
- SW4 pad 2: GND -> +5V
- SW40 pad 2: GND -> +5V
- SW41 pad 2: GND -> +5V
- SW42 pad 2: GND -> +5V
- SW43 pad 2: GND -> +5V
- SW44 pad 2: GND -> +5V
- SW45 pad 2: GND -> +5V
- SW46 pad 2: GND -> +5V
- SW46 pad 3: COL1 -> COL0
- SW47 pad 2: GND -> +5V
- SW47 pad 3: COL0 -> COL1
- SW48 pad 2: GND -> +5V
- SW49 pad 2: GND -> +5V
- SW5 pad 2: GND -> +5V
- SW50 pad 2: GND -> +5V
- SW51 pad 2: GND -> +5V
- SW52 pad 2: GND -> +5V
- SW53 pad 2: GND -> +5V
- SW54 pad 2: GND -> +5V
- SW55 pad 2: GND -> +5V
- SW56 pad 2: GND -> +5V
- SW57 pad 2: GND -> +5V
- SW58 pad 2: GND -> +5V
- SW59 pad 2: GND -> +5V
- SW6 pad 2: GND -> +5V
- SW60 pad 2: GND -> +5V
- SW61 pad 2: GND -> +5V
- SW62 pad 2: GND -> +5V
- SW63 pad 2: GND -> +5V
- SW64 pad 2: GND -> +5V
- SW65 pad 2: GND -> +5V
- SW66 pad 2: GND -> +5V
- SW67 pad 2: GND -> +5V
- SW68 pad 2: GND -> +5V
- SW69 pad 2: GND -> +5V
- SW7 pad 2: GND -> +5V
- SW70 pad 2: GND -> +5V
- SW71 pad 2: GND -> +5V
- SW72 pad 2: GND -> +5V
- SW72 pad 3: COL0 -> COL1
- SW73 pad 2: GND -> +5V
- SW73 pad 3: COL1 -> COL0
- SW74 pad 2: GND -> +5V
- SW75 pad 2: GND -> +5V
- SW76 pad 2: GND -> +5V
- SW77 pad 2: GND -> +5V
- SW78 pad 2: GND -> +5V
- SW79 pad 2: GND -> +5V
- SW8 pad 2: GND -> +5V
- SW80 pad 2: GND -> +5V
- SW81 pad 2: GND -> +5V
- SW82 pad 2: GND -> +5V
- SW83 pad 2: GND -> +5V
- SW84 pad 2: GND -> +5V
- SW85 pad 2: GND -> +5V
- SW86 pad 2: GND -> +5V
- SW87 pad 2: GND -> +5V
- SW88 pad 2: GND -> +5V
- SW89 pad 2: GND -> +5V
- SW9 pad 2: GND -> +5V
- SW90 pad 2: GND -> +5V
- SW91 pad 2: GND -> +5V
- SW92 pad 2: GND -> +5V
- SW93 pad 2: GND -> +5V
- SW94 pad 2: GND -> +5V
- SW95 pad 2: GND -> +5V
- SW96 pad 2: GND -> +5V
- SW96 pad 3: COL0 -> COL1
- SW97 pad 2: GND -> +5V
- SW97 pad 3: COL1 -> COL0
- SW98 pad 2: GND -> +5V
- SW99 pad 2: GND -> +5V
- U1 pad 14: /COL12 -> COL12
- U1 pad 15: /COL13 -> COL13
- U1 pad 16: /COL14 -> COL14
- U1 pad 17: /COL15 -> COL15
- U1 pad 6: COL5 -> /COL5
- U1 pad 7: COL6 -> /COL6
- U1 pad 8: COL7 -> /COL7
- U2 pad 2: Net-(C13-Pad1) -> /X1
- U2 pad 22: /ROW1 -> ROW1
- U2 pad 23: /ROW2 -> ROW2
- U2 pad 24: /ROW3 -> ROW3
- U2 pad 3: Net-(C14-Pad1) -> /X2
- U2 pad 35: /ROW4 -> ROW4
- U2 pad 37: /ROW6 -> ROW6
- U2 pad 38: /ROW7 -> ROW7
Routing:
- net +5V: track 0.00 -> 3684.0 mm, vias 0 -> 26
- net ROW7: track 0.00 -> 989.6 mm, vias 0 -> 9
- net COL1: track 61.6 -> 1046.0 mm, vias 0 -> 17
- net GND: track 15.3 -> 966.6 mm, vias 0 -> 27
- net COL0: track 72.2 -> 990.7 mm, vias 0 -> 17
- net COL3: track 69.8 -> 948.5 mm, vias 0 -> 15
- net COL2: track 71.9 -> 942.6 mm, vias 0 -> 17
- net ROW5: track 19.1 -> 815.9 mm, vias 0 -> 8
- net COL5: track 75.6 -> 860.5 mm, vias 0 -> 12
- net ROW0: track 59.1 -> 827.4 mm, vias 0 -> 21
- net COL4: track 79.0 -> 799.3 mm, vias 0 -> 21
- net COL6: track 69.7 -> 743.3 mm, vias 0 -> 12
- net COL7: track 71.1 -> 712.4 mm, vias 0 -> 18
- net ROW3: track 0.00 -> 544.5 mm
- net ROW2: track 0.00 -> 521.4 mm
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
Commit message: Done modern routing.
Parts:
- moved JP24 2.25 mm to (476.1, 121.2)
- moved JP23 2.18 mm to (476.1, 124.6)
Connections:
- U1 pad 10: /COL9 -> COL9
- U1 pad 11: /COL10 -> COL10
- U1 pad 13: /COL11 -> COL11
- U1 pad 6: /COL5 -> COL5
- U1 pad 7: /COL6 -> COL6
- U1 pad 8: /COL7 -> COL7
- U1 pad 9: /COL8 -> COL8
Routing:
- net ROW4: track 500.7 -> 585.9 mm, vias 0 -> 2
- net COL2: track 942.6 -> 953.0 mm
- net COL0: track 990.7 -> 984.2 mm
- net COL12: track 349.0 -> 344.7 mm, vias 15 -> 14
- net READ: track 93.2 -> 90.9 mm
- net CONN27: track 45.4 -> 47.7 mm
- net CONN29: track 53.5 -> 51.7 mm
- net INT: track 94.2 -> 96.0 mm
- net COL1: track 1046.0 -> 1045.0 mm
- net ROW5: track 815.9 -> 815.0 mm
- net ROW3: track 544.5 -> 543.7 mm
- net ROW2: track 521.4 -> 520.7 mm
- net COL7: track 712.4 -> 711.7 mm
- net RESET: track 169.2 -> 168.5 mm
- net GND: track 966.6 -> 966.0 mm
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
Commit message: Updated the rounded variant.
Parts:
- removed ? (x28): , 
- removed the REF** at (340.6, 108.5)
- removed the REF** at (340.6, 96.0)
- added C12: 10pF, TestPoint:Two_Pad_Through_Hole_10.4mm, F.Cu at (230.7, 104.9)
- added C13: 10pF, TestPoint:Two_Pad_Through_Hole_10.4mm, F.Cu at (301.6, 114.8)
- added C14: 10pF, TestPoint:Two_Pad_Through_Hole_10.4mm, F.Cu at (301.6, 117.9)
- added C15: 15pF, TestPoint:Two_Pad_Through_Hole_10.4mm, F.Cu at (524.6, 111.2)
- added C16: 22uF 15v, TestPoint:Two_Pad_Through_Hole_20mm, F.Cu at (515.7, 117.0)
- added C17: 4.7uF 25v, TestPoint:Two_Pad_Through_Hole_12mm, F.Cu at (509.8, 111.6)
- added R10: 1K, TestPoint:Two_Pad_Through_Hole_12.4mm, F.Cu at (422.0, 92.4)
- added R11: 1K, TestPoint:Two_Pad_Through_Hole_12.4mm, F.Cu at (419.5, 89.8)
- added R4: 1K, TestPoint:Two_Pad_Through_Hole_12.4mm, F.Cu at (340.6, 102.2)
- added R5: 1K, TestPoint:Two_Pad_Through_Hole_12.4mm, F.Cu at (343.9, 102.2)
- added R6: 1K, TestPoint:Two_Pad_Through_Hole_12.4mm, F.Cu at (383.8, 98.0)
- added R7: 1K, TestPoint:Two_Pad_Through_Hole_12.4mm, F.Cu at (389.0, 95.8)
- added R8: 1K, TestPoint:Two_Pad_Through_Hole_12.4mm, F.Cu at (402.4, 98.0)
- added R9: 1K, TestPoint:Two_Pad_Through_Hole_12.4mm, F.Cu at (419.5, 94.9)
- added Y3: Crystal 3.58MHz, TestPoint:Two_Pad_Through_Hole_10.4mm, F.Cu at (301.8, 111.5)
Connections:
- U1 pad 10: COL9 -> /COL9
- U1 pad 11: COL10 -> /COL10
- U1 pad 13: COL11 -> /COL11
- U1 pad 14: COL12 -> /COL12
- U1 pad 15: COL13 -> /COL13
- U1 pad 16: COL14 -> /COL14
- U1 pad 17: COL15 -> /COL15
- U1 pad 4: COL3 -> /COL3
- U1 pad 6: COL5 -> /COL5
- U1 pad 7: COL6 -> /COL6
- U1 pad 8: COL7 -> /COL7
- U1 pad 9: COL8 -> /COL8
Routing:
- net GND: track 966.0 -> 1018.8 mm
- net ROW4: track 585.9 -> 587.9 mm
- net +5V: track 3684.3 -> 3685.5 mm
- net ROW5: track 815.0 -> 816.0 mm
- net ROW3: track 543.7 -> 542.9 mm
Other:
- board text added: "Trace extends to the edge of the board. -->"
