File: SpaceCadet.kicad_pcb (KiCad board)
At the start: 2 copper layers, 469 x 166.6 mm, 202 parts, among them J0 Conn_02x17_Odd_Even, J3_1 Conn_01x04, J3_2 Conn_01x04, SW1 SD_4B3E, SW10 SD_4B3E, SW100 SD_4B3E, SW101 SD_4B3E, SW102 SD_4B3E, SW103 SD_4B3E, SW104 SD_4B3E, SW105 SD_4B3E, SW106 SD_4B3E, SW107 SD_4B3E, SW108 SD_4B3E, SW109 SD_4B3E, SW11 SD_4B3E, SW110 SD_4B3E, SW111 SD_4B3E, SW112 SD_4B3E, SW113 SD_4B3E, SW114 SD_4B3E, SW115 SD_4B3E, SW116 SD_4B3E, SW117 SD_4B3E, SW118 SD_4B3E, SW119 SD_4B3E, SW12 SD_4B3E, SW120 SD_4B3E, SW121 SD_4B3E, SW122 SD_4B3E, SW122a0 SD_4B3E, SW123 SD_4B3E, SW123a0 SD_4B3E, SW124 SD_4B3E, SW124a0 SD_4B3E, SW125 SD_4B3E, SW126 SD_4B3E, SW127 SD_4B3E, SW128 SD_4B3E, SW13 SD_4B3E, SW14 SD_4B3E, SW15 SD_4B3E, SW16 SD_4B3E, SW17 SD_4B3E, SW18 SD_4B3E, SW19 SD_4B3E, SW2 SD_4B3E, SW20 SD_4B3E, SW21 SD_4B3E, SW22 SD_4B3E, SW23 SD_4B3E, SW24 SD_4B3E, SW25 SD_4B3E, SW26 SD_4B3E, SW27 SD_4B3E, SW28 SD_4B3E, SW29 SD_4B3E, SW3 SD_4B3E, SW30 SD_4B3E, SW31 SD_4B3E, SW32 SD_4B3E, SW33 SD_4B3E, SW34 SD_4B3E, SW35 SD_4B3E, SW36 SD_4B3E, SW37 SD_4B3E, SW38 SD_4B3E, SW39 SD_4B3E, SW4 SD_4B3E, SW40 SD_4B3E, SW41 SD_4B3E, SW42 SD_4B3E, SW43 SD_4B3E, SW44 SD_4B3E, SW45 SD_4B3E, SW46 SD_4B3E, SW47 SD_4B3E, SW48 SD_4B3E, SW49 SD_4B3E, SW5 SD_4B3E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

Commit message: Brought over bug fixes from other branch. Fixed some paths to be closer to original. Fixed path going through mount hole.
Parts:
- removed the ? at (526.4, 117.1)
- removed the ? at (497.7, 111.1)
- removed the ? at (382.8, 95.6)
- removed the ? at (425.6, 94.7)
- removed the ? at (230.8, 99.9)
- removed the ? at (413.6, 94.7)
- removed the ? at (425.4, 89.7)
- removed the ? at (416.3, 92.3)
- removed the ? at (307.0, 111.6)
- removed the ? at (296.4, 114.8)
- removed the ? at (390.1, 98.0)
- removed the ? at (395.2, 95.6)
- removed the ? at (516.4, 111.1)
- removed the ? at (306.7, 114.8)
- removed the ? at (306.7, 117.9)
- removed the ? at (343.9, 108.5)
- removed the ? at (519.3, 111.1)
- removed the ? at (501.0, 117.1)
- removed the ? at (343.9, 96.0)
- removed the ? at (413.6, 89.7)
- removed the ? at (230.8, 110.2)
- removed the ? at (529.6, 111.1)
- removed the ? at (396.2, 98.0)
- removed the ? at (377.7, 98.0)
- removed the ? at (408.7, 98.0)
- removed the ? at (296.4, 117.9)
- removed the ? at (296.6, 111.6)
- removed the ? at (428.1, 92.3)
- removed the REF** at (340.6, 108.5)
- removed the REF** at (340.6, 96.0)
- added ?: ThroughHole, ThroughHole, F.Cu at (365.9, 179.1)
- added ?: ThroughHole, ThroughHole, F.Cu at (412.8, 236.6)
- added ?: ThroughHole, ThroughHole, F.Cu at (198.1, 189.6)
- added ?: ThroughHole, ThroughHole, F.Cu at (127.6, 186.1)
- added ?: ThroughHole, ThroughHole, F.Cu at (275.4, 112.3)
- added ?: ThroughHole, ThroughHole, F.Cu at (109.1, 104.5)
- added ?: ThroughHole, ThroughHole, F.Cu at (151.3, 216.3)
- added ?: ThroughHole, ThroughHole, F.Cu at (318.8, 148.5)
- added ?: ThroughHole, ThroughHole, F.Cu at (379.5, 227.6)
- added ?: ThroughHole, ThroughHole, F.Cu at (296.5, 114.8)
- added ?: ThroughHole, ThroughHole, F.Cu at (416.2, 92.5)
- added ?: ThroughHole, ThroughHole, F.Cu at (428.0, 92.5)
- added ?: ThroughHole, ThroughHole, F.Cu at (451.7, 196.4)
- added ?: ThroughHole, ThroughHole, F.Cu at (375.1, 160.6)
- added ?: ThroughHole, ThroughHole, F.Cu at (275.2, 186.4)
- added ?: ThroughHole, ThroughHole, F.Cu at (197.9, 200.0)
- added ?: ThroughHole, ThroughHole, F.Cu at (228.0, 216.6)
- added ?: ThroughHole, ThroughHole, F.Cu at (322.5, 202.2)
- added ?: ThroughHole, ThroughHole, F.Cu at (440.0, 110.7)
- added ?: ThroughHole, ThroughHole, F.Cu at (516.2, 111.1)
- added ?: ThroughHole, ThroughHole, F.Cu at (313.3, 197.1)
- added ?: ThroughHole, ThroughHole, F.Cu at (471.4, 237.9)
- added ?: ThroughHole, ThroughHole, F.Cu at (436.0, 88.5)
- added ?: ThroughHole, ThroughHole, F.Cu at (70.5, 142.6)
- added ?: ThroughHole, ThroughHole, F.Cu at (318.8, 161.5)
- added ?: ThroughHole, ThroughHole, F.Cu at (488.9, 176.8)
- added ?: ThroughHole, ThroughHole, F.Cu at (395.5, 156.4)
- added ?: ThroughHole, ThroughHole, F.Cu at (451.9, 110.9)
- added ?: ThroughHole, ThroughHole, F.Cu at (488.9, 157.6)
- added ?: ThroughHole, ThroughHole, F.Cu at (183.8, 154.5)
- added ?: ThroughHole, ThroughHole, F.Cu at (352.1, 199.0)
- added ?: ThroughHole, ThroughHole, F.Cu at (350.0, 117.9)
- added ?: ThroughHole, ThroughHole, F.Cu at (246.8, 216.3)
- added ?: ThroughHole, ThroughHole, F.Cu at (346.3, 178.5)
- added ?: ThroughHole, ThroughHole, F.Cu at (329.1, 168.6)
- added ?: ThroughHole, ThroughHole, F.Cu at (164.9, 148.1)
- added ?: ThroughHole, ThroughHole, F.Cu at (395.2, 95.7)
- added ?: ThroughHole, ThroughHole, F.Cu at (363.1, 164.9)
- added ?: ThroughHole, ThroughHole, F.Cu at (229.4, 100.1)
- added ?: ThroughHole, ThroughHole, F.Cu at (501.0, 117.0)
- added ?: ThroughHole, ThroughHole, F.Cu at (313.6, 114.0)
- added ?: ThroughHole, ThroughHole, F.Cu at (185.6, 143.3)
- added ?: ThroughHole, ThroughHole, F.Cu at (469.2, 171.4)
- added ?: ThroughHole, ThroughHole, F.Cu at (81.5, 87.5)
- added ?: ThroughHole, ThroughHole, F.Cu at (442.7, 104.0)
- added ?: ThroughHole, ThroughHole, F.Cu at (122.1, 126.1)
- added ?: ThroughHole, ThroughHole, F.Cu at (359.8, 204.5)
- added ?: ThroughHole, ThroughHole, F.Cu at (142.3, 110.6)
- added ?: ThroughHole, ThroughHole, F.Cu at (135.0, 104.5)
- added ?: ThroughHole, ThroughHole, F.Cu at (164.9, 162.5)
- added ?: ThroughHole, ThroughHole, F.Cu at (361.4, 230.3)
- added ?: ThroughHole, ThroughHole, F.Cu at (428.2, 186.4)
- added ?: ThroughHole, ThroughHole, F.Cu at (148.1, 119.6)
- added ?: ThroughHole, ThroughHole, F.Cu at (170.6, 224.5)
- added ?: ThroughHole, ThroughHole, F.Cu at (222.6, 150.5)
- added ?: ThroughHole, ThroughHole, F.Cu at (306.6, 111.7)
- added ?: ThroughHole, ThroughHole, F.Cu at (242.2, 163.1)
- added ?: ThroughHole, ThroughHole, F.Cu at (378.7, 145.2)
- added ?: ThroughHole, ThroughHole, F.Cu at (170.3, 215.4)
- added ?: ThroughHole, ThroughHole, F.Cu at (134.5, 89.2)
- added ?: ThroughHole, ThroughHole, F.Cu at (101.3, 89.2)
- added ?: ThroughHole, ThroughHole, F.Cu at (332.5, 104.0)
- added ?: ThroughHole, ThroughHole, F.Cu at (275.2, 197.3)
- added ?: ThroughHole, ThroughHole, F.Cu at (469.6, 198.1)
- added ?: ThroughHole, ThroughHole, F.Cu at (413.6, 138.8)
- added ?: ThroughHole, ThroughHole, F.Cu at (356.2, 106.5)
- added ?: ThroughHole, ThroughHole, F.Cu at (346.3, 167.0)
- added ?: ThroughHole, ThroughHole, F.Cu at (89.5, 184.3)
- added ?: ThroughHole, ThroughHole, F.Cu at (440.6, 229.8)
- added ?: ThroughHole, ThroughHole, F.Cu at (193.3, 181.6)
- added ?: ThroughHole, ThroughHole, F.Cu at (135.9, 108.0)
- added ?: ThroughHole, ThroughHole, F.Cu at (146.0, 104.5)
- added ?: ThroughHole, ThroughHole, F.Cu at (490.6, 216.2)
- added ?: ThroughHole, ThroughHole, F.Cu at (142.3, 120.2)
- added ?: ThroughHole, ThroughHole, F.Cu at (261.4, 149.1)
- added ?: ThroughHole, ThroughHole, F.Cu at (362.7, 202.0)
- added ?: ThroughHole, ThroughHole, F.Cu at (451.6, 106.4)
- added ?: ThroughHole, ThroughHole, F.Cu at (359.8, 217.0)
- added ?: ThroughHole, ThroughHole, F.Cu at (393.6, 142.3)
- added ?: ThroughHole, ThroughHole, F.Cu at (94.9, 100.8)
- added ?: ThroughHole, ThroughHole, F.Cu at (130.6, 146.2)
- added ?: ThroughHole, ThroughHole, F.Cu at (203.5, 148.9)
- added ?: ThroughHole, ThroughHole, F.Cu at (341.6, 216.6)
- added ?: ThroughHole, ThroughHole, F.Cu at (232.5, 169.0)
- added ?: ThroughHole, ThroughHole, F.Cu at (406.7, 240.2)
- added ?: ThroughHole, ThroughHole, F.Cu at (119.5, 104.5)
- added ?: ThroughHole, ThroughHole, F.Cu at (425.4, 94.9)
- added ?: ThroughHole, ThroughHole, F.Cu at (89.5, 214.1)
- added ?: ThroughHole, ThroughHole, F.Cu at (428.0, 120.9)
- added ?: ThroughHole, ThroughHole, F.Cu at (326.1, 165.0)
- added ?: ThroughHole, ThroughHole, F.Cu at (192.2, 202.7)
- added ?: ThroughHole, ThroughHole, F.Cu at (122.9, 110.6)
- added ?: ThroughHole, ThroughHole, F.Cu at (145.9, 129.5)
- added ?: ThroughHole, ThroughHole, F.Cu at (175.3, 167.1)
- added ?: ThroughHole, ThroughHole, F.Cu at (86.6, 146.2)
- added ?: ThroughHole, ThroughHole, F.Cu at (451.7, 215.8)
- added ?: ThroughHole, ThroughHole, F.Cu at (148.1, 100.7)
- added ?: ThroughHole, ThroughHole, F.Cu at (237.2, 198.6)
- added ?: ThroughHole, ThroughHole, F.Cu at (242.2, 132.4)
- added ?: ThroughHole, ThroughHole, F.Cu at (131.9, 104.5)
- added ?: ThroughHole, ThroughHole, F.Cu at (251.7, 178.6)
- added ?: ThroughHole, ThroughHole, F.Cu at (359.3, 117.9)
- added ?: ThroughHole, ThroughHole, F.Cu at (490.6, 203.0)
- added ?: ThroughHole, ThroughHole, F.Cu at (151.3, 236.8)
- added ?: ThroughHole, ThroughHole, F.Cu at (112.1, 89.4)
- added ?: ThroughHole, ThroughHole, F.Cu at (439.3, 120.9)
- added ?: ThroughHole, ThroughHole, F.Cu at (332.5, 117.3)
- added ?: ThroughHole, ThroughHole, F.Cu at (488.9, 198.8)
- added ?: ThroughHole, ThroughHole, F.Cu at (141.3, 126.1)
- added ?: ThroughHole, ThroughHole, F.Cu at (127.6, 157.8)
- added ?: ThroughHole, ThroughHole, F.Cu at (91.7, 100.8)
- added ?: ThroughHole, ThroughHole, F.Cu at (222.6, 130.7)
- added ?: ThroughHole, ThroughHole, F.Cu at (284.4, 216.5)
- added ?: ThroughHole, ThroughHole, F.Cu at (261.4, 163.6)
- added ?: ThroughHole, ThroughHole, F.Cu at (296.5, 111.7)
- added ?: ThroughHole, ThroughHole, F.Cu at (329.1, 179.6)
- added ?: ThroughHole, ThroughHole, F.Cu at (108.7, 165.6)
- added ?: ThroughHole, ThroughHole, F.Cu at (422.5, 98.1)
- added ?: ThroughHole, ThroughHole, F.Cu at (370.3, 196.2)
- added ?: ThroughHole, ThroughHole, F.Cu at (70.5, 179.1)
- added ?: ThroughHole, ThroughHole, F.Cu at (377.6, 98.0)
- added ?: ThroughHole, ThroughHole, F.Cu at (337.2, 144.5)
- added ?: ThroughHole, ThroughHole, F.Cu at (103.9, 110.9)
- added ?: ThroughHole, ThroughHole, F.Cu at (418.3, 213.3)
- added ?: ThroughHole, ThroughHole, F.Cu at (284.4, 203.5)
- added ?: ThroughHole, ThroughHole, F.Cu at (483.8, 117.7)
- added ?: ThroughHole, ThroughHole, F.Cu at (119.9, 90.0)
- added ?: ThroughHole, ThroughHole, F.Cu at (509.0, 157.5)
- added ?: ThroughHole, ThroughHole, F.Cu at (278.9, 157.0)
- added ?: ThroughHole, ThroughHole, F.Cu at (313.6, 104.0)
- added ?: ThroughHole, ThroughHole, F.Cu at (125.2, 126.1)
- added ?: ThroughHole, ThroughHole, F.Cu at (289.9, 178.3)
- added ?: ThroughHole, ThroughHole, F.Cu at (406.7, 228.9)
- added ?: ThroughHole, ThroughHole, F.Cu at (370.5, 183.8)
- added ?: ThroughHole, ThroughHole, F.Cu at (236.9, 186.3)
- added ?: ThroughHole, ThroughHole, F.Cu at (164.9, 129.4)
- added ?: ThroughHole, ThroughHole, F.Cu at (164.9, 151.5)
- added ?: ThroughHole, ThroughHole, F.Cu at (346.8, 117.3)
- added ?: ThroughHole, ThroughHole, F.Cu at (139.2, 95.5)
- added ?: ThroughHole, ThroughHole, F.Cu at (75.0, 146.2)
- added ?: ThroughHole, ThroughHole, F.Cu at (355.2, 145.5)
- added ?: ThroughHole, ThroughHole, F.Cu at (270.7, 178.4)
- added ?: ThroughHole, ThroughHole, F.Cu at (376.9, 125.2)
- added ?: ThroughHole, ThroughHole, F.Cu at (203.5, 129.4)
- added ?: ThroughHole, ThroughHole, F.Cu at (195.5, 202.7)
- added ?: ThroughHole, ThroughHole, F.Cu at (332.5, 107.3)
- added ?: ThroughHole, ThroughHole, F.Cu at (306.6, 114.8)
- added ?: ThroughHole, ThroughHole, F.Cu at (509.1, 210.5)
- added ?: ThroughHole, ThroughHole, F.Cu at (356.2, 117.9)
- added ?: ThroughHole, ThroughHole, F.Cu at (361.4, 211.4)
- added ?: ThroughHole, ThroughHole, F.Cu at (526.4, 117.0)
- added ?: ThroughHole, ThroughHole, F.Cu at (265.8, 203.6)
- added ?: ThroughHole, ThroughHole, F.Cu at (413.6, 157.5)
- added ?: ThroughHole, ThroughHole, F.Cu at (89.5, 165.8)
- added ?: ThroughHole, ThroughHole, F.Cu at (246.8, 203.4)
- added ?: ThroughHole, ThroughHole, F.Cu at (341.6, 202.8)
- added ?: ThroughHole, ThroughHole, F.Cu at (242.2, 151.9)
- added ?: ThroughHole, ThroughHole, F.Cu at (148.9, 194.5)
- added ?: ThroughHole, ThroughHole, F.Cu at (337.2, 162.8)
- added ?: ThroughHole, ThroughHole, F.Cu at (261.4, 152.1)
- added ?: ThroughHole, ThroughHole, F.Cu at (472.4, 196.0)
- added ?: ThroughHole, ThroughHole, F.Cu at (185.6, 147.0)
- added ?: ThroughHole, ThroughHole, F.Cu at (313.6, 110.6)
- added ?: ThroughHole, ThroughHole, F.Cu at (127.6, 237.1)
- added ?: ThroughHole, ThroughHole, F.Cu at (127.8, 101.4)
- added ?: ThroughHole, ThroughHole, F.Cu at (108.7, 195.5)
- added ?: ThroughHole, ThroughHole, F.Cu at (471.4, 138.9)
- added ?: ThroughHole, ThroughHole, F.Cu at (101.3, 100.8)
- added ?: ThroughHole, ThroughHole, F.Cu at (89.5, 139.1)
- added ?: ThroughHole, ThroughHole, F.Cu at (306.6, 117.9)
- added ?: ThroughHole, ThroughHole, F.Cu at (109.0, 89.4)
- added ?: ThroughHole, ThroughHole, F.Cu at (151.3, 202.7)
- added ?: ThroughHole, ThroughHole, F.Cu at (355.2, 163.6)
- added ?: ThroughHole, ThroughHole, F.Cu at (109.0, 100.7)
- added ?: ThroughHole, ThroughHole, F.Cu at (313.5, 120.4)
- added ?: ThroughHole, ThroughHole, F.Cu at (382.7, 95.7)
- added ?: ThroughHole, ThroughHole, F.Cu at (469.6, 211.0)
- added ?: ThroughHole, ThroughHole, F.Cu at (98.1, 89.2)
- added ?: ThroughHole, ThroughHole, F.Cu at (228.0, 204.0)
- added ?: ThroughHole, ThroughHole, F.Cu at (142.3, 113.8)
- added ?: ThroughHole, ThroughHole, F.Cu at (488.9, 138.9)
- added ?: ThroughHole, ThroughHole, F.Cu at (281.1, 130.4)
- added ?: ThroughHole, ThroughHole, F.Cu at (78.1, 104.5)
- added ?: ThroughHole, ThroughHole, F.Cu at (303.6, 216.5)
- added ?: ThroughHole, ThroughHole, F.Cu at (89.5, 203.0)
- added ?: ThroughHole, ThroughHole, F.Cu at (343.8, 108.5)
- added ?: ThroughHole, ThroughHole, F.Cu at (451.7, 139.1)
- added ?: ThroughHole, ThroughHole, F.Cu at (451.7, 157.5)
- added ?: ThroughHole, ThroughHole, F.Cu at (141.3, 146.2)
- added ?: ThroughHole, ThroughHole, F.Cu at (156.5, 178.2)
- added ?: ThroughHole, ThroughHole, F.Cu at (332.5, 114.0)
- added ?: ThroughHole, ThroughHole, F.Cu at (89.5, 176.1)
- added ?: ThroughHole, ThroughHole, F.Cu at (91.7, 89.2)
- added ?: ThroughHole, ThroughHole, F.Cu at (389.3, 198.9)
- added ?: ThroughHole, ThroughHole, F.Cu at (509.0, 139.2)
- added ?: ThroughHole, ThroughHole, F.Cu at (471.4, 157.5)
- added ?: ThroughHole, ThroughHole, F.Cu at (160.6, 186.3)
- added ?: ThroughHole, ThroughHole, F.Cu at (313.6, 101.0)
- added ?: ThroughHole, ThroughHole, F.Cu at (94.9, 89.2)
- added ?: ThroughHole, ThroughHole, F.Cu at (131.0, 89.2)
- added ?: ThroughHole, ThroughHole, F.Cu at (469.2, 153.0)
- added ?: ThroughHole, ThroughHole, F.Cu at (411.7, 98.1)
- added ?: ThroughHole, ThroughHole, F.Cu at (478.9, 120.2)
- added ?: ThroughHole, ThroughHole, F.Cu at (448.4, 178.1)
- added ?: ThroughHole, ThroughHole, F.Cu at (412.8, 225.3)
- added ?: ThroughHole, ThroughHole, F.Cu at (265.6, 216.5)
- added ?: ThroughHole, ThroughHole, F.Cu at (124.9, 101.4)
- added ?: ThroughHole, ThroughHole, F.Cu at (281.1, 161.0)
- added ?: ThroughHole, ThroughHole, F.Cu at (112.1, 100.7)
- added ?: ThroughHole, ThroughHole, F.Cu at (290.1, 167.7)
- added ?: ThroughHole, ThroughHole, F.Cu at (331.8, 186.4)
- added ?: ThroughHole, ThroughHole, F.Cu at (108.7, 218.9)
- added ?: ThroughHole, ThroughHole, F.Cu at (122.9, 120.2)
- added ?: ThroughHole, ThroughHole, F.Cu at (359.3, 106.5)
- added ?: ThroughHole, ThroughHole, F.Cu at (151.3, 233.6)
- added ?: ThroughHole, ThroughHole, F.Cu at (436.0, 118.2)
- added ?: ThroughHole, ThroughHole, F.Cu at (119.9, 101.4)
- added ?: ThroughHole, ThroughHole, F.Cu at (218.8, 186.6)
- added ?: ThroughHole, ThroughHole, F.Cu at (399.0, 233.6)
- added ?: ThroughHole, ThroughHole, F.Cu at (246.8, 239.4)
- added ?: ThroughHole, ThroughHole, F.Cu at (108.7, 157.8)
- added ?: ThroughHole, ThroughHole, F.Cu at (529.5, 111.1)
- added ?: ThroughHole, ThroughHole, F.Cu at (332.5, 101.0)
- added ?: ThroughHole, ThroughHole, F.Cu at (309.2, 167.4)
- added ?: ThroughHole, ThroughHole, F.Cu at (116.7, 108.0)
- added ?: ThroughHole, ThroughHole, F.Cu at (332.5, 110.6)
- added ?: ThroughHole, ThroughHole, F.Cu at (376.6, 203.3)
- added ?: ThroughHole, ThroughHole, F.Cu at (193.6, 170.4)
- added ?: ThroughHole, ThroughHole, F.Cu at (185.6, 157.7)
- added ?: ThroughHole, ThroughHole, F.Cu at (122.9, 113.8)
- added ?: ThroughHole, ThroughHole, F.Cu at (78.3, 87.5)
- added ?: ThroughHole, ThroughHole, F.Cu at (440.6, 211.2)
- added ?: ThroughHole, ThroughHole, F.Cu at (365.6, 203.3)
- added ?: ThroughHole, ThroughHole, F.Cu at (229.4, 110.2)
- added ?: ThroughHole, ThroughHole, F.Cu at (256.2, 186.4)
- added ?: ThroughHole, ThroughHole, F.Cu at (373.8, 182.2)
- added ?: ThroughHole, ThroughHole, F.Cu at (518.7, 106.9)
- added ?: ThroughHole, ThroughHole, F.Cu at (213.2, 167.6)
- added ?: ThroughHole, ThroughHole, F.Cu at (413.6, 94.9)
- added ?: ThroughHole, ThroughHole, F.Cu at (299.1, 150.5)
- added ?: ThroughHole, ThroughHole, F.Cu at (116.7, 110.9)
- added ?: ThroughHole, ThroughHole, F.Cu at (428.2, 197.7)
- added ?: ThroughHole, ThroughHole, F.Cu at (89.5, 195.2)
- added ?: ThroughHole, ThroughHole, F.Cu at (350.0, 106.5)
- added ?: ThroughHole, ThroughHole, F.Cu at (296.5, 117.9)
- added ?: ThroughHole, ThroughHole, F.Cu at (145.9, 148.7)
- added ?: ThroughHole, ThroughHole, F.Cu at (317.0, 144.3)
- added ?: ThroughHole, ThroughHole, F.Cu at (451.7, 199.5)
- added ?: ThroughHole, ThroughHole, F.Cu at (365.9, 168.6)
- added ?: ThroughHole, ThroughHole, F.Cu at (207.9, 228.4)
- added ?: ThroughHole, ThroughHole, F.Cu at (218.8, 198.7)
- added ?: ThroughHole, ThroughHole, F.Cu at (364.0, 121.1)
- added ?: ThroughHole, ThroughHole, F.Cu at (324.2, 115.3)
- added ?: ThroughHole, ThroughHole, F.Cu at (509.1, 228.5)
- added ?: ThroughHole, ThroughHole, F.Cu at (170.3, 204.4)
- added ?: ThroughHole, ThroughHole, F.Cu at (134.5, 100.7)
- added ?: ThroughHole, ThroughHole, F.Cu at (89.5, 217.6)
- added ?: ThroughHole, ThroughHole, F.Cu at (381.8, 164.9)
- added ?: ThroughHole, ThroughHole, F.Cu at (313.3, 186.7)
- added ?: ThroughHole, ThroughHole, F.Cu at (175.3, 178.3)
- added ?: ThroughHole, ThroughHole, F.Cu at (303.4, 203.9)
- added ?: ThroughHole, ThroughHole, F.Cu at (75.1, 87.5)
- added ?: ThroughHole, ThroughHole, F.Cu at (89.5, 233.7)
- added ?: ThroughHole, ThroughHole, F.Cu at (471.4, 217.6)
- added ?: ThroughHole, ThroughHole, F.Cu at (376.1, 121.1)
- added ?: ThroughHole, ThroughHole, F.Cu at (497.9, 111.1)
- added ?: ThroughHole, ThroughHole, F.Cu at (322.5, 214.6)
- added ?: ThroughHole, ThroughHole, F.Cu at (488.9, 211.0)
- added ?: ThroughHole, ThroughHole, F.Cu at (108.7, 176.0)
- added ?: ThroughHole, ThroughHole, F.Cu at (393.6, 161.1)
- added ?: ThroughHole, ThroughHole, F.Cu at (150.6, 95.6)
- added ?: ThroughHole, ThroughHole, F.Cu at (171.1, 236.8)
- added ?: ThroughHole, ThroughHole, F.Cu at (81.5, 99.0)
- added ?: ThroughHole, ThroughHole, F.Cu at (317.0, 126.2)
- added ?: ThroughHole, ThroughHole, F.Cu at (472.4, 179.4)
- added ?: ThroughHole, ThroughHole, F.Cu at (379.5, 208.4)
- added ?: ThroughHole, ThroughHole, F.Cu at (200.4, 186.3)
- added ?: ThroughHole, ThroughHole, F.Cu at (127.6, 220.3)
- added ?: ThroughHole, ThroughHole, F.Cu at (313.6, 107.3)
- added ?: ThroughHole, ThroughHole, F.Cu at (160.6, 198.6)
- added ?: ThroughHole, ThroughHole, F.Cu at (353.1, 106.5)
- added ?: ThroughHole, ThroughHole, F.Cu at (196.0, 167.4)
- added ?: ThroughHole, ThroughHole, F.Cu at (408.6, 98.1)
- added ?: ThroughHole, ThroughHole, F.Cu at (189.8, 215.8)
- added ?: ThroughHole, ThroughHole, F.Cu at (108.7, 146.2)
- added ?: ThroughHole, ThroughHole, F.Cu at (393.7, 182.2)
- added ?: ThroughHole, ThroughHole, F.Cu at (171.0, 233.2)
- added ?: ThroughHole, ThroughHole, F.Cu at (97.5, 104.5)
- added ?: ThroughHole, ThroughHole, F.Cu at (89.5, 157.8)
- added ?: ThroughHole, ThroughHole, F.Cu at (70.5, 198.7)
- added ?: ThroughHole, ThroughHole, F.Cu at (213.2, 178.6)
- added ?: ThroughHole, ThroughHole, F.Cu at (326.1, 176.8)
- added ?: ThroughHole, ThroughHole, F.Cu at (350.2, 196.1)
- added ?: ThroughHole, ThroughHole, F.Cu at (71.9, 87.5)
- added ?: ThroughHole, ThroughHole, F.Cu at (346.8, 106.0)
- added ?: ThroughHole, ThroughHole, F.Cu at (116.5, 90.0)
- added ?: ThroughHole, ThroughHole, F.Cu at (433.1, 138.9)
- added ?: ThroughHole, ThroughHole, F.Cu at (318.8, 130.9)
- added ?: ThroughHole, ThroughHole, F.Cu at (207.9, 209.2)
- added ?: ThroughHole, ThroughHole, F.Cu at (355.2, 133.9)
- added ?: ThroughHole, ThroughHole, F.Cu at (335.2, 115.3)
- added ?: ThroughHole, ThroughHole, F.Cu at (213.2, 202.7)
- added ?: ThroughHole, ThroughHole, F.Cu at (413.6, 89.7)
- added ?: ThroughHole, ThroughHole, F.Cu at (467.7, 120.2)
- added ?: ThroughHole, ThroughHole, F.Cu at (359.8, 145.2)
- added ?: ThroughHole, ThroughHole, F.Cu at (440.0, 107.0)
- added ?: ThroughHole, ThroughHole, F.Cu at (375.1, 149.7)
- added ?: ThroughHole, ThroughHole, F.Cu at (396.1, 98.1)
- added ?: ThroughHole, ThroughHole, F.Cu at (294.1, 186.2)
- added ?: ThroughHole, ThroughHole, F.Cu at (261.4, 132.2)
- added ?: ThroughHole, ThroughHole, F.Cu at (339.8, 228.6)
- added ?: ThroughHole, ThroughHole, F.Cu at (299.1, 160.8)
- added ?: ThroughHole, ThroughHole, F.Cu at (122.9, 117.0)
- added ?: ThroughHole, ThroughHole, F.Cu at (179.8, 198.6)
- added ?: ThroughHole, ThroughHole, F.Cu at (185.6, 127.7)
- added ?: ThroughHole, ThroughHole, F.Cu at (313.6, 117.3)
- added ?: ThroughHole, ThroughHole, F.Cu at (127.8, 90.0)
- added ?: ThroughHole, ThroughHole, F.Cu at (246.8, 221.0)
- added ?: ThroughHole, ThroughHole, F.Cu at (294.2, 197.3)
- added ?: ThroughHole, ThroughHole, F.Cu at (200.4, 198.1)
- added ?: ThroughHole, ThroughHole, F.Cu at (179.8, 186.7)
- added ?: ThroughHole, ThroughHole, F.Cu at (448.4, 199.5)
- added ?: ThroughHole, ThroughHole, F.Cu at (222.6, 147.4)
- added ?: ThroughHole, ThroughHole, F.Cu at (71.9, 99.0)
- added ?: ThroughHole, ThroughHole, F.Cu at (433.1, 157.5)
- added ?: ThroughHole, ThroughHole, F.Cu at (299.1, 146.9)
- added ?: ThroughHole, ThroughHole, F.Cu at (203.5, 145.7)
- added ?: ThroughHole, ThroughHole, F.Cu at (370.5, 187.0)
- added ?: ThroughHole, ThroughHole, F.Cu at (488.9, 216.2)
- added ?: ThroughHole, ThroughHole, F.Cu at (309.2, 178.5)
- added ?: ThroughHole, ThroughHole, F.Cu at (70.5, 160.6)
- added ?: ThroughHole, ThroughHole, F.Cu at (148.9, 213.5)
- added ?: ThroughHole, ThroughHole, F.Cu at (418.3, 202.1)
- added ?: ThroughHole, ThroughHole, F.Cu at (381.8, 202.0)
- added ?: ThroughHole, ThroughHole, F.Cu at (281.1, 150.4)
- added ?: ThroughHole, ThroughHole, F.Cu at (337.2, 133.1)
- added ?: ThroughHole, ThroughHole, F.Cu at (232.6, 178.4)
- added ?: ThroughHole, ThroughHole, F.Cu at (124.9, 90.0)
- added ?: ThroughHole, ThroughHole, F.Cu at (389.0, 183.8)
- added ?: ThroughHole, ThroughHole, F.Cu at (242.2, 148.9)
- added ?: ThroughHole, ThroughHole, F.Cu at (203.5, 159.8)
- added ?: ThroughHole, ThroughHole, F.Cu at (436.0, 99.8)
- added ?: ThroughHole, ThroughHole, F.Cu at (270.7, 167.8)
- added ?: ThroughHole, ThroughHole, F.Cu at (145.9, 145.7)
- added ?: ThroughHole, ThroughHole, F.Cu at (145.9, 227.1)
- added ?: ThroughHole, ThroughHole, F.Cu at (210.3, 205.2)
- added ?: ThroughHole, ThroughHole, F.Cu at (519.4, 111.1)
- added ?: ThroughHole, ThroughHole, F.Cu at (78.3, 99.0)
- added ?: ThroughHole, ThroughHole, F.Cu at (318.8, 141.3)
- added ?: ThroughHole, ThroughHole, F.Cu at (183.8, 135.7)
- added ?: ThroughHole, ThroughHole, F.Cu at (103.8, 126.1)
- added ?: ThroughHole, ThroughHole, F.Cu at (189.8, 204.5)
- added ?: ThroughHole, ThroughHole, F.Cu at (340.6, 108.5)
- added ?: ThroughHole, ThroughHole, F.Cu at (488.9, 230.5)
- added ?: ThroughHole, ThroughHole, F.Cu at (131.0, 100.7)
- added ?: ThroughHole, ThroughHole, F.Cu at (127.6, 182.5)
- added ?: ThroughHole, ThroughHole, F.Cu at (353.1, 117.9)
- added ?: ThroughHole, ThroughHole, F.Cu at (127.6, 217.5)
- added ?: ThroughHole, ThroughHole, F.Cu at (127.6, 201.9)
- added ?: ThroughHole, ThroughHole, F.Cu at (454.1, 100.9)
- added ?: ThroughHole, ThroughHole, F.Cu at (281.1, 147.2)
- added ?: ThroughHole, ThroughHole, F.Cu at (251.7, 167.8)
- added ?: ThroughHole, ThroughHole, F.Cu at (142.3, 117.0)
- added ?: ThroughHole, ThroughHole, F.Cu at (339.8, 209.5)
- added ?: ThroughHole, ThroughHole, F.Cu at (70.5, 163.9)
- added ?: ThroughHole, ThroughHole, F.Cu at (98.1, 100.8)
- added ?: ThroughHole, ThroughHole, F.Cu at (195.7, 178.2)
- added ?: ThroughHole, ThroughHole, F.Cu at (286.5, 112.3)
- added ?: ThroughHole, ThroughHole, F.Cu at (399.0, 214.6)
- added ?: ThroughHole, ThroughHole, F.Cu at (472.4, 117.7)
- added ?: ThroughHole, ThroughHole, F.Cu at (145.9, 208.0)
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Routing:
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
Commit message: Checkpoint
Connections:
- ? pad : (no net) -> COL3 (x4)
- ? pad : (no net) -> COL14 (x4)
- ? pad : (no net) -> COL11 (x6)
- ? pad : (no net) -> COL6 (x6)
- ? pad : (no net) -> CONN9
- ? pad : (no net) -> GND (x17)
- ? pad : (no net) -> COL5 (x4)
- ? pad : (no net) -> COL4 (x7)
- ? pad : (no net) -> COL9 (x5)
- ? pad : (no net) -> COL10 (x6)
- ? pad : (no net) -> CONN5
- ? pad : (no net) -> COL8 (x2)
- ? pad : (no net) -> COL2 (x8)
- ? pad : (no net) -> CONN2
- ? pad : (no net) -> COL0 (x3)
- ? pad : (no net) -> COL13 (x3)
- ? pad : (no net) -> ROW4
- ? pad : (no net) -> COL12 (x7)
- ? pad : (no net) -> A5 (x2)
- ? pad : (no net) -> COL7 (x2)
- ? pad : (no net) -> ROW3
- ? pad : (no net) -> ROW0
- ? pad : (no net) -> ROW7
- ? pad : (no net) -> COL1 (x3)
- U1 pad 15: /COL13 -> COL13
- U2 pad 24: /ROW3 -> ROW3
- U2 pad 26: +5V -> GND
- U2 pad 35: /ROW4 -> ROW4
- U2 pad 37: /ROW6 -> COL6
Routing:
- net (no net): track 193.5 -> 3959.1 mm
- net GND: track 15.3 -> 3696.0 mm
- net COL6: track 70.5 -> 843.5 mm
- net COL3: track 69.8 -> 797.6 mm
- net COL5: track 76.1 -> 789.7 mm
- net COL2: track 71.9 -> 763.1 mm
- net COL0: track 72.2 -> 721.0 mm
- net COL1: track 61.6 -> 706.3 mm
- net ROW4: track 0.00 -> 570.0 mm
- net ROW0: track 59.1 -> 606.9 mm
- net ROW3: track 0.00 -> 539.1 mm
- net CONN10: track 0.00 -> 424.7 mm
- net CONN8: track 0.00 -> 400.6 mm
- net ROW7: track 0.00 -> 396.1 mm
- net CONN6: track 0.00 -> 384.3 mm
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
Commit message: Minor edits
Parts:
- moved ? 1.46 mm to (230.8, 100.1)
- moved ? 1.46 mm to (230.8, 110.2)
Changed lines of the file:
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@@
   )
   (footprint "ThroughHole" (layer "F.Cu")
-    (at 229.39 100.09 90)
+    (at 230.85 100.09 90)
     (attr through_hole)
     (fp_text reference "" (at 0 0 90) (layer "F.SilkS")
@@
   )
   (footprint "ThroughHole" (layer "F.Cu")
-    (at 229.39 110.15 90)
+    (at 230.85 110.15 90)
     (attr through_hole)
     (fp_text reference "" (at 0 0 90) (layer "F.SilkS")
@@
   (arc (start 337.184946 108.29916) (mid 337.878506 109.184269) (end 338.6817 109.971242) (width 0.25) (layer "B.Cu") (net 47))
   (arc (start 391.563808 104.305845) (mid 390.660692 105.018295) (end 389.730659 105.695231) (width 0.25) (layer "B.Cu") (net 47))
-  (segment (start 218.628936 101.233463) (end 220.873781 100.908247) (width 0.25) (layer "B.Cu") (net 48))
-  (segment (start 228.49888 100.572732) (end 225.529832 100.572732) (width 0.25) (layer "B.Cu") (net 48))
+  (segment (start 218.695738 100.800421) (end 220.940583 100.475205) (width 0.25) (layer "B.Cu") (net 48))
+  (segment (start 228.565682 100.13969) (end 225.596634 100.13969) (width 0.25) (layer "B.Cu") (net 48))
   (segment (start 356.97724 102.674993) (end 357.277285 102.642298) (width 0.25) (layer "B.Cu") (net 48))
-  (segment (start 214.069728 102.234963) (end 210.033955 103.433099) (width 0.25) (layer "B.Cu") (net 48))
+  (segment (start 214.13653 101.801921) (end 210.100757 103.000057) (width 0.25) (layer "B.Cu") (net 48))
   (segment (start 351.281001 105.126198) (end 350.396545 106.571706) (width 0.25) (layer "B.Cu") (net 48))
-  (segment (start 233.116276 101.076894) (end 238.565507 102.281231) (width 0.25) (layer "B.Cu") (net 48))
-  (segment (start 204.146384 104.627341) (end 205.474768 104.434787) (width 0.25) (layer "B.Cu") (net 48))
+  (segment (start 233.183078 100.643852) (end 238.632309 101.848189) (width 0.25) (layer "B.Cu") (net 48))
+  (segment (start 204.213186 104.194299) (end 205.54157 104.001745) (width 0.25) (layer "B.Cu") (net 48))
   (segment (start 379.630597 121.338778) (end 381.151298 117.341284) (width 0.25) (layer "B.Cu") (net 48))
   (segment (start 360.760999 102.41744) (end 370.631485 102.21632) (width 0.25) (layer "B.Cu") (net 48))
-  (segment (start 199.490367 104.963042) (end 145.653198 104.963042) (width 0.25) (layer "B.Cu") (net 48))
+  (segment (start 199.557169 104.53) (end 145.72 104.53) (width 0.25) (layer "B.Cu") (net 48))
   (segment (start 354.152209 103.234081) (end 353.446241 103.438785) (width 0.25) (layer "B.Cu") (net 48))
   (arc (start 378.595075 123.238305) (mid 377.896959 124.068857) (end 377.098144 124.803076) (width 0.25) (layer "B.Cu") (net 48))
-  (arc (start 204.146384 104.627341) (mid 201.824418 104.879007) (end 199.490367 104.963042) (width 0.25) (layer "B.Cu") (net 48))
-  (arc (start 233.116276 101.076894) (mid 230.821299 100.699145) (end 228.49888 100.572732) (width 0.25) (layer "B.Cu") (net 48))
+  (arc (start 204.213186 104.194299) (mid 201.89122 104.445965) (end 199.557169 104.53) (width 0.25) (layer "B.Cu") (net 48))
+  (arc (start 233.183078 100.643852) (mid 230.888101 100.266103) (end 228.565682 100.13969) (width 0.25) (layer "B.Cu") (net 48))
   (arc (start 360.760999 102.41744) (mid 359.016663 102.491469) (end 357.277285 102.642298) (width 0.25) (layer "B.Cu") (net 48))
-  (arc (start 225.529832 100.572732) (mid 223.19577 100.656719) (end 220.873781 100.908247) (width 0.25) (layer "B.Cu") (net 48))
-  (arc (start 210.033955 103.433099) (mid 207.77248 104.016408) (end 205.474768 104.434787) (width 0.25) (layer "B.Cu") (net 48))
+  (arc (start 225.596634 100.13969) (mid 223.262572 100.223677) (end 220.940583 100.475205) (width 0.25) (layer "B.Cu") (net 48))
+  (arc (start 210.100757 103.000057) (mid 207.839282 103.583366) (end 205.54157 104.001745) (width 0.25) (layer "B.Cu") (net 48))
   (arc (start 353.446241 103.438785) (mid 352.795846 103.69819) (end 352.207879 104.078453) (width 0.25) (layer "B.Cu") (net 48))
   (arc (start 356.97724 102.674993) (mid 355.552579 102.893166) (end 354.152209 103.234081) (width 0.25) (layer "B.Cu") (net 48))
   (arc (start 352.207879 104.078453) (mid 351.69844 104.561632) (end 351.281001 105.126198) (width 0.25) (layer "B.Cu") (net 48))
   (arc (start 379.630597 121.338778) (mid 379.177329 122.3237) (end 378.595075 123.238305) (width 0.25) (layer "B.Cu") (net 48))
-  (arc (start 218.628936 101.233463) (mid 216.331207 101.651701) (end 214.069728 102.234963) (width 0.25) (layer "B.Cu") (net 48))
+  (arc (start 218.695738 100.800421) (mid 216.398009 101.218659) (end 214.13653 101.801921) (width 0.25) (layer "B.Cu") (net 48))
   (segment (start 364.479406 121.05003) (end 371.091154 117.821767) (width 0.25) (layer "B.Cu") (net 49))
   (segment (start 371.261491 120.055991) (end 373.904551 117.27849) (width 0.25) (layer "B.Cu") (net 50))
@@
     )
   )
-  (group "" (id 41118133-1dd3-45a3-bfa0-4f4588c514e9)
-    (members
-      561ce965-2595-427c-ada4-57937b00c127
-      b8d06d02-13ad-4d49-9a9e-2611d489794b
-    )
-  )

Commit message: Added traces, jumpers to front to use DRC. Fixed lots of real and imaginary DRC errors/warnings.
Parts:
- removed the ? at (109.1, 104.5)
- added JP18: Jumper Open, Jumper:SolderJumper-2_P1.3mm_Open_TrianglePad1.0x1.5mm, F.Cu at (346.7, 111.9)
- added JP19: Jumper Open, Jumper:SolderJumper-2_P1.3mm_Open_TrianglePad1.0x1.5mm, F.Cu at (369.7, 121.2)
- added JP20: Jumper Bridged, Jumper:SolderJumper-2_P1.3mm_Bridged2Bar_Pad1.0x1.5mm, F.Cu at (445.9, 110.8)
- added JP21: Jumper Bridged, Jumper:SolderJumper-2_P1.3mm_Bridged2Bar_Pad1.0x1.5mm, F.Cu at (445.9, 106.7)
- added JP22: Jumper Bridged, Jumper:SolderJumper-2_P1.3mm_Bridged2Bar_Pad1.0x1.5mm, F.Cu at (448.2, 103.9)
- added JP23: Jumper Open, Jumper:SolderJumper-2_P1.3mm_Open_TrianglePad1.0x1.5mm, F.Cu at (473.3, 120.5)
- added JP24: Jumper Bridged, Jumper:SolderJumper-2_P1.3mm_Bridged2Bar_Pad1.0x1.5mm, F.Cu at (477.5, 117.5)
- added JP25: Jumper Open, Jumper:SolderJumper-2_P1.3mm_Open_TrianglePad1.0x1.5mm, F.Cu at (75.2, 93.9)
- added JP26: Jumper Open, Jumper:SolderJumper-2_P1.3mm_Open_TrianglePad1.0x1.5mm, F.Cu at (81.7, 93.1)
- added JP27: Jumper Open, Jumper:SolderJumper-2_P1.3mm_Open_TrianglePad1.0x1.5mm, F.Cu at (94.8, 94.7)
- added JP28: Jumper Open, Jumper:SolderJumper-2_P1.3mm_Open_TrianglePad1.0x1.5mm, F.Cu at (98.1, 94.8)
- added JP29: Jumper Open, Jumper:SolderJumper-2_P1.3mm_Open_TrianglePad1.0x1.5mm, F.Cu at (112.2, 95.3)
- added JP30: Jumper Open, Jumper:SolderJumper-2_P1.3mm_Open_TrianglePad1.0x1.5mm, F.Cu at (119.8, 96.0)
- added JP31: Jumper Open, Jumper:SolderJumper-2_P1.3mm_Open_TrianglePad1.0x1.5mm, F.Cu at (124.8, 95.9)
- added JP32: Jumper Open, Jumper:SolderJumper-2_P1.3mm_Open_TrianglePad1.0x1.5mm, F.Cu at (134.3, 95.8)
- moved ? 1.76 mm to (471.4, 236.1)
- moved ? 1.35 mm to (70.7, 162.6)
- moved ? 1.31 mm to (70.7, 181.2)
- moved ? 0.92 mm to (183.8, 134.8)
- moved ? 0.76 mm to (509.1, 229.3)
- moved ? 0.73 mm to (89.5, 214.8)
- moved ? 0.66 mm to (170.9, 204.4)
- moved ? 0.63 mm to (242.2, 133.1)
- moved ? 0.60 mm to (170.9, 215.4)
- moved ? 0.56 mm to (108.7, 176.6)
- moved ? 0.54 mm to (210.3, 220.1)
- moved ? 0.53 mm to (440.0, 106.4)
- moved ? 0.52 mm to (326.1, 165.6)
- moved ? 0.50 mm to (379.5, 228.1)
- moved ? 0.49 mm to (469.2, 152.5)
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Connections:
- ? pad : (no net) -> COL13 (x15)
- ? pad : (no net) -> +5V (x22)
- ? pad : (no net) -> ROW0 (x21)
- ? pad : (no net) -> COL3 (x12)
- ? pad : (no net) -> GND (x31)
- ? pad : (no net) -> ROW6 (x3)
- ? pad : (no net) -> ROW1
- ? pad : COL6 -> ROW6 (x2)
- ? pad : (no net) -> COL10 (x8)
- ? pad : (no net) -> COL7 (x14)
- ? pad : (no net) -> COL12 (x7)
- ? pad : (no net) -> WRITE
- ? pad : (no net) -> COL6 (x8)
- ? pad : (no net) -> COL1 (x14)
- ? pad : (no net) -> COL9 (x9)
- ? pad : (no net) -> COL5 (x8)
- ? pad : (no net) -> COL15 (x16)
- ? pad : (no net) -> COL8 (x8)
- ? pad : (no net) -> /A0 (x2)
- ? pad : GND -> +5V (x7)
- ? pad : (no net) -> A6 (x3)
- ? pad : (no net) -> COL14 (x10)
- ? pad : (no net) -> /X1 (x4)
- ? pad : (no net) -> CONN4
- ? pad : (no net) -> /A3 (x2)
- ? pad : (no net) -> ROW5 (x9)
- ? pad : (no net) -> COL0 (x14)
- ? pad : (no net) -> ROW7 (x9)
- ? pad : (no net) -> COL4 (x14)
- ? pad : (no net) -> A5 (x2)
- ? pad : (no net) -> CONN6
- ? pad : (no net) -> /X2 (x4)
- ? pad : (no net) -> CONN27
- ? pad : (no net) -> COL11 (x8)
- ? pad : (no net) -> /A2 (x2)
- ? pad : (no net) -> /A1 (x2)
- ? pad : (no net) -> COL2 (x9)
- ? pad : (no net) -> CONN8
- ? pad : (no net) -> /A4 (x2)
- ? pad : (no net) -> CONN29
- ? pad : (no net) -> ROW2
- ? pad : (no net) -> T0
- ? pad : (no net) -> CONN10
- ? pad : COL0 -> COL1
- ? pad : (no net) -> CONN33
- ? pad : (no net) -> RESET
- ? pad : (no net) -> A7 (x3)
- ? pad : (no net) -> T1
- ? pad : (no net) -> INT
- ? pad : (no net) -> ROW4 (x2)
- ? pad : (no net) -> READ
- ? pad : (no net) -> CONN3
- ? pad : COL1 -> COL0
- J3_1 pad 1: COL0 -> ROW0
- J3_1 pad 2: COL1 -> ROW1
- J3_1 pad 3: COL2 -> ROW2
- J3_1 pad 4: COL3 -> ROW3
- J3_2 pad 1: COL4 -> ROW4
- J3_2 pad 2: COL5 -> ROW5
- J3_2 pad 3: COL6 -> ROW6
- J3_2 pad 4: COL7 -> ROW7
- SW1 pad 2: GND -> +5V
- SW10 pad 2: GND -> +5V
- SW100 pad 2: GND -> +5V
- SW101 pad 2: GND -> +5V
- SW102 pad 2: GND -> +5V
- SW103 pad 2: GND -> +5V
- SW104 pad 2: GND -> +5V
- SW105 pad 2: GND -> +5V
- SW106 pad 2: GND -> +5V
- SW107 pad 2: GND -> +5V
- SW108 pad 2: GND -> +5V
- SW109 pad 2: GND -> +5V
- SW11 pad 2: GND -> +5V
- SW110 pad 2: GND -> +5V
- SW111 pad 2: GND -> +5V
- SW112 pad 2: GND -> +5V
- SW113 pad 2: GND -> +5V
- SW114 pad 2: GND -> +5V
- SW115 pad 2: GND -> +5V
- SW116 pad 2: GND -> +5V
- SW117 pad 2: GND -> +5V
- SW118 pad 2: GND -> +5V
- SW119 pad 2: GND -> +5V
- SW119 pad 3: COL0 -> COL1
- SW12 pad 2: GND -> +5V
- SW120 pad 2: GND -> +5V
- SW120 pad 3: COL1 -> COL0
- SW121 pad 2: GND -> +5V
- SW122 pad 2: GND -> +5V
- SW122a0 pad 2: GND -> +5V
- SW123 pad 2: GND -> +5V
- SW123a0 pad 2: GND -> +5V
- SW124 pad 2: GND -> +5V
- SW124a0 pad 2: GND -> +5V
- SW125 pad 2: GND -> +5V
- SW126 pad 2: GND -> +5V
- SW127 pad 2: GND -> +5V
- SW128 pad 2: GND -> +5V
- SW13 pad 2: GND -> +5V
- SW14 pad 2: GND -> +5V
- SW15 pad 2: GND -> +5V
- SW16 pad 2: GND -> +5V
- SW17 pad 2: GND -> +5V
- SW18 pad 2: GND -> +5V
- SW19 pad 2: GND -> +5V
- SW2 pad 2: GND -> +5V
- SW2 pad 3: unconnected-(SW2-Pad3) -> COL1
- SW20 pad 2: GND -> +5V
- SW21 pad 2: GND -> +5V
- SW22 pad 2: GND -> +5V
- SW22 pad 3: COL1 -> COL0
- SW23 pad 2: GND -> +5V
- SW23 pad 3: COL0 -> COL1
- SW24 pad 2: GND -> +5V
- SW25 pad 2: GND -> +5V
- SW26 pad 2: GND -> +5V
- SW27 pad 2: GND -> +5V
- SW28 pad 2: GND -> +5V
- SW29 pad 2: GND -> +5V
- SW3 pad 2: GND -> +5V
- SW3 pad 3: unconnected-(SW3-Pad3) -> COL0
- SW30 pad 2: GND -> +5V
- SW31 pad 2: GND -> +5V
- SW32 pad 2: GND -> +5V
- SW33 pad 2: GND -> +5V
- SW34 pad 2: GND -> +5V
- SW35 pad 2: GND -> +5V
- SW36 pad 2: GND -> +5V
- SW37 pad 2: GND -> +5V
- SW38 pad 2: GND -> +5V
- SW39 pad 2: GND -> +5V
- SW4 pad 2: GND -> +5V
- SW40 pad 2: GND -> +5V
- SW41 pad 2: GND -> +5V
- SW42 pad 2: GND -> +5V
- SW43 pad 2: GND -> +5V
- SW44 pad 2: GND -> +5V
- SW45 pad 2: GND -> +5V
- SW46 pad 2: GND -> +5V
- SW46 pad 3: COL1 -> COL0
- SW47 pad 2: GND -> +5V
- SW47 pad 3: COL0 -> COL1
- SW48 pad 2: GND -> +5V
- SW49 pad 2: GND -> +5V
- SW5 pad 2: GND -> +5V
- SW50 pad 2: GND -> +5V
- SW51 pad 2: GND -> +5V
- SW52 pad 2: GND -> +5V
- SW53 pad 2: GND -> +5V
- SW54 pad 2: GND -> +5V
- SW55 pad 2: GND -> +5V
- SW56 pad 2: GND -> +5V
- SW57 pad 2: GND -> +5V
- SW58 pad 2: GND -> +5V
- SW59 pad 2: GND -> +5V
- SW6 pad 2: GND -> +5V
- SW60 pad 2: GND -> +5V
- SW61 pad 2: GND -> +5V
- SW62 pad 2: GND -> +5V
- SW63 pad 2: GND -> +5V
- SW64 pad 2: GND -> +5V
- SW65 pad 2: GND -> +5V
- SW66 pad 2: GND -> +5V
- SW67 pad 2: GND -> +5V
- SW68 pad 2: GND -> +5V
- SW69 pad 2: GND -> +5V
- SW7 pad 2: GND -> +5V
- SW70 pad 2: GND -> +5V
- SW71 pad 2: GND -> +5V
- SW72 pad 2: GND -> +5V
- SW72 pad 3: COL0 -> COL1
- SW73 pad 2: GND -> +5V
- SW73 pad 3: COL1 -> COL0
- SW74 pad 2: GND -> +5V
- SW75 pad 2: GND -> +5V
- SW76 pad 2: GND -> +5V
- SW77 pad 2: GND -> +5V
- SW78 pad 2: GND -> +5V
- SW79 pad 2: GND -> +5V
- SW8 pad 2: GND -> +5V
- SW80 pad 2: GND -> +5V
- SW81 pad 2: GND -> +5V
- SW82 pad 2: GND -> +5V
- SW83 pad 2: GND -> +5V
- SW84 pad 2: GND -> +5V
- SW85 pad 2: GND -> +5V
- SW86 pad 2: GND -> +5V
- SW87 pad 2: GND -> +5V
- SW88 pad 2: GND -> +5V
- SW89 pad 2: GND -> +5V
- SW9 pad 2: GND -> +5V
- SW90 pad 2: GND -> +5V
- SW91 pad 2: GND -> +5V
- SW92 pad 2: GND -> +5V
- SW93 pad 2: GND -> +5V
- SW94 pad 2: GND -> +5V
- SW95 pad 2: GND -> +5V
- SW96 pad 2: GND -> +5V
- SW96 pad 3: COL0 -> COL1
- SW97 pad 2: GND -> +5V
- SW97 pad 3: COL1 -> COL0
- SW98 pad 2: GND -> +5V
- SW99 pad 2: GND -> +5V
- U1 pad 15: COL13 -> /COL13
- U1 pad 4: COL3 -> /COL3
- U1 pad 6: COL5 -> /COL5
- U1 pad 7: COL6 -> /COL6
- U1 pad 8: COL7 -> /COL7
- U2 pad 2: Net-(C13-Pad1) -> /X1
- U2 pad 22: /ROW1 -> ROW1
- U2 pad 23: /ROW2 -> ROW2
- U2 pad 26: GND -> +5V
- U2 pad 3: Net-(C14-Pad1) -> /X2
- U2 pad 37: COL6 -> ROW6
- U2 pad 38: /ROW7 -> ROW7
Routing:
- net (no net): track 3959.1 -> 0.00 mm
- net +5V: track 123.9 -> 3716.6 mm
- net GND: track 3696.0 -> 1033.6 mm
- net ROW5: track 148.5 -> 811.9 mm
- net ROW7: track 396.1 -> 1001.0 mm
- net ROW2: track 0.00 -> 514.6 mm
- net COL4: track 463.8 -> 854.6 mm
- net COL1: track 706.3 -> 1068.0 mm
- net COL7: track 351.7 -> 697.9 mm
- net ROW1: track 193.5 -> 491.2 mm
- net COL0: track 721.0 -> 1005.5 mm
- net ROW0: track 606.9 -> 828.8 mm
- net COL2: track 763.1 -> 970.8 mm
- net ROW6: track 363.8 -> 551.6 mm
- net COL3: track 797.6 -> 965.8 mm
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
Commit message: Now one-sided board.
Parts:
- removed JP18, JP19, JP23, JP25, JP26, JP27, JP28, JP29, JP30, JP31, JP32: Jumper Open, Jumper:SolderJumper-2_P1.3mm_Open_TrianglePad1.0x1.5mm
- removed JP20, JP21, JP22, JP24: Jumper Bridged, Jumper:SolderJumper-2_P1.3mm_Bridged2Bar_Pad1.0x1.5mm
Routing:
- net GND: track 1033.6 -> 837.8 mm
- net +5V: track 3716.6 -> 3530.2 mm
- net ROW0: track 828.8 -> 687.5 mm
- net COL4: track 854.6 -> 717.3 mm
- net COL1: track 1068.0 -> 933.3 mm
- net COL3: track 965.8 -> 842.1 mm
- net COL0: track 1005.5 -> 882.5 mm
- net COL13: track 513.5 -> 390.7 mm
- net COL15: track 440.1 -> 322.8 mm
- net COL2: track 970.8 -> 854.8 mm
- net COL7: track 697.9 -> 586.5 mm
- net COL11: track 329.3 -> 232.8 mm
- net COL12: track 323.9 -> 228.4 mm
- net COL9: track 410.5 -> 317.7 mm
- net COL10: track 367.2 -> 274.8 mm
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Other:
- board text added: "* Copper only on the BACK side. Through-hole plating is not required. * Solder mask only on BACK side. * Silkscreen only on the FRONT side."
- board text added: "Reproduction of historic hand-drawn board."
- board text added: "Track extends to edge of the board at this point. ——>"
