File: SpaceCadet.kicad_pcb (KiCad board)
At the start: 2 copper layers, 469 x 166.6 mm, 581 parts, among them J0 Conn_02x17_Odd_Even, J3_1 Conn_01x04, J3_2 Conn_01x04, SW1 SD_4B3E, SW10 SD_4B3E, SW100 SD_4B3E, SW101 SD_4B3E, SW102 SD_4B3E, SW103 SD_4B3E, SW104 SD_4B3E, SW105 SD_4B3E, SW106 SD_4B3E, SW107 SD_4B3E, SW108 SD_4B3E, SW109 SD_4B3E, SW11 SD_4B3E, SW110 SD_4B3E, SW111 SD_4B3E, SW112 SD_4B3E, SW113 SD_4B3E, SW114 SD_4B3E, SW115 SD_4B3E, SW116 SD_4B3E, SW117 SD_4B3E, SW118 SD_4B3E, SW119 SD_4B3E, SW12 SD_4B3E, SW120 SD_4B3E, SW121 SD_4B3E, SW122 SD_4B3E, SW122a0 SD_4B3E, SW123 SD_4B3E, SW123a0 SD_4B3E, SW124 SD_4B3E, SW124a0 SD_4B3E, SW125 SD_4B3E, SW126 SD_4B3E, SW127 SD_4B3E, SW128 SD_4B3E, SW13 SD_4B3E, SW14 SD_4B3E, SW15 SD_4B3E, SW16 SD_4B3E, SW17 SD_4B3E, SW18 SD_4B3E, SW19 SD_4B3E, SW2 SD_4B3E, SW20 SD_4B3E, SW21 SD_4B3E, SW22 SD_4B3E, SW23 SD_4B3E, SW24 SD_4B3E, SW25 SD_4B3E, SW26 SD_4B3E, SW27 SD_4B3E, SW28 SD_4B3E, SW29 SD_4B3E, SW3 SD_4B3E, SW30 SD_4B3E, SW31 SD_4B3E, SW32 SD_4B3E, SW33 SD_4B3E, SW34 SD_4B3E, SW35 SD_4B3E, SW36 SD_4B3E, SW37 SD_4B3E, SW38 SD_4B3E, SW39 SD_4B3E, SW4 SD_4B3E, SW40 SD_4B3E, SW41 SD_4B3E, SW42 SD_4B3E, SW43 SD_4B3E, SW44 SD_4B3E, SW45 SD_4B3E, SW46 SD_4B3E, SW47 SD_4B3E, SW48 SD_4B3E, SW49 SD_4B3E, SW5 SD_4B3E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

Commit message: Added front-side copper for constraint check. Debugged switch footprint.
Parts:
- removed the ? at (296.5, 114.8)
- removed the ? at (416.2, 92.5)
- removed the ? at (428.0, 92.5)
- removed the ? at (516.2, 111.1)
- removed the ? at (395.2, 95.7)
- removed the ? at (230.8, 100.1)
- removed the ? at (501.0, 117.0)
- removed the ? at (306.6, 111.7)
- removed the ? at (425.4, 94.9)
- removed the ? at (296.5, 111.7)
- removed the ? at (377.6, 98.0)
- removed the ? at (306.6, 114.8)
- removed the ? at (526.4, 117.0)
- removed the ? at (306.6, 117.9)
- removed the ? at (382.7, 95.7)
- removed the ? at (343.8, 108.5)
- removed the ? at (529.5, 111.1)
- removed the ? at (230.8, 110.2)
- removed the ? at (413.6, 94.9)
- removed the ? at (296.5, 117.9)
- removed the ? at (497.9, 111.1)
- removed the ? at (408.6, 98.1)
- removed the ? at (413.6, 89.7)
- removed the ? at (396.1, 98.1)
- removed the ? at (519.4, 111.1)
- removed the ? at (340.6, 108.5)
- removed the ? at (340.6, 96.0)
- removed the ? at (425.4, 89.7)
- removed the ? at (390.0, 98.0)
- removed the ? at (343.8, 96.0)
- added C12: 10pF, TestPoint:Two_Pad_Through_Hole_10.4mm, F.Cu at (230.7, 105.2)
- added C13: 10pF, TestPoint:Two_Pad_Through_Hole_10.4mm, F.Cu at (301.6, 114.7)
- added C14: 10pF, TestPoint:Two_Pad_Through_Hole_10.4mm, F.Cu at (301.6, 117.8)
- added C15: 15pF, TestPoint:Two_Pad_Through_Hole_10.4mm, F.Cu at (524.2, 111.0)
- added C16: 22uF 15v, TestPoint:Two_Pad_Through_Hole_20mm, F.Cu at (513.7, 117.1)
- added C17: 4.7uF 25v, TestPoint:Two_Pad_Through_Hole_12mm, F.Cu at (507.5, 111.1)
- added JP18: Jumper Open, Jumper:SolderJumper-2_P1.3mm_Open_TrianglePad1.0x1.5mm, F.Cu at (346.8, 111.5)
- added JP19: Jumper Open, Jumper:SolderJumper-2_P1.3mm_Open_TrianglePad1.0x1.5mm, F.Cu at (367.3, 121.1)
- added JP20: Jumper Bridged, Jumper:SolderJumper-2_P1.3mm_Bridged2Bar_Pad1.0x1.5mm, F.Cu at (445.8, 110.8)
- added JP21: Jumper Bridged, Jumper:SolderJumper-2_P1.3mm_Bridged2Bar_Pad1.0x1.5mm, F.Cu at (445.8, 106.4)
- added JP22: Jumper Bridged, Jumper:SolderJumper-2_P1.3mm_Bridged2Bar_Pad1.0x1.5mm, F.Cu at (445.9, 103.8)
- added JP23: Jumper Open, Jumper:SolderJumper-2_P1.3mm_Open_TrianglePad1.0x1.5mm, F.Cu at (475.0, 120.3)
- added JP24: Jumper Bridged, Jumper:SolderJumper-2_P1.3mm_Bridged2Bar_Pad1.0x1.5mm, F.Cu at (475.9, 117.7)
- added JP25: Jumper Open, Jumper:SolderJumper-2_P1.3mm_Open_TrianglePad1.0x1.5mm, F.Cu at (75.2, 95.5)
- added JP26: Jumper Open, Jumper:SolderJumper-2_P1.3mm_Open_TrianglePad1.0x1.5mm, F.Cu at (81.6, 95.5)
- added JP27: Jumper Open, Jumper:SolderJumper-2_P1.3mm_Open_TrianglePad1.0x1.5mm, F.Cu at (95.0, 97.9)
- added JP28: Jumper Open, Jumper:SolderJumper-2_P1.3mm_Open_TrianglePad1.0x1.5mm, F.Cu at (98.1, 97.9)
- added JP29: Jumper Open, Jumper:SolderJumper-2_P1.3mm_Open_TrianglePad1.0x1.5mm, F.Cu at (112.1, 97.7)
- added JP30: Jumper Open, Jumper:SolderJumper-2_P1.3mm_Open_TrianglePad1.0x1.5mm, F.Cu at (119.9, 98.0)
- added JP31: Jumper Open, Jumper:SolderJumper-2_P1.3mm_Open_TrianglePad1.0x1.5mm, F.Cu at (124.9, 98.0)
- added JP32: Jumper Open, Jumper:SolderJumper-2_P1.3mm_Open_TrianglePad1.0x1.5mm, F.Cu at (134.4, 97.5)
- added R10: 1K, TestPoint:Two_Pad_Through_Hole_12.4mm, F.Cu at (422.0, 92.3)
- added R11: 1K, TestPoint:Two_Pad_Through_Hole_12.4mm, F.Cu at (419.5, 89.7)
- added R4: 1K, TestPoint:Two_Pad_Through_Hole_12.4mm, F.Cu at (340.6, 102.2)
- added R5: 1K, TestPoint:Two_Pad_Through_Hole_12.4mm, F.Cu at (343.9, 102.2)
- added R6: 1K, TestPoint:Two_Pad_Through_Hole_12.4mm, F.Cu at (383.8, 97.8)
- added R7: 1K, TestPoint:Two_Pad_Through_Hole_12.4mm, F.Cu at (389.0, 95.7)
- added R8: 1K, TestPoint:Two_Pad_Through_Hole_12.4mm, F.Cu at (402.4, 97.9)
- added R9: 1K, TestPoint:Two_Pad_Through_Hole_12.4mm, F.Cu at (419.5, 94.8)
- added Y3: Crystal 3.58MHz, TestPoint:Two_Pad_Through_Hole_10.4mm, F.Cu at (301.8, 111.5)
Routing:
- net COL15: track 322.8 -> 539.9 mm
- net GND: track 837.8 -> 1042.6 mm
- net +5V: track 3530.2 -> 3716.6 mm
- net COL5: track 700.0 -> 875.5 mm
- net COL7: track 586.5 -> 758.9 mm
- net COL14: track 184.8 -> 343.8 mm
- net COL6: track 613.3 -> 770.7 mm
- net COL12: track 228.4 -> 376.2 mm
- net COL0: track 882.5 -> 1021.9 mm
- net COL4: track 717.3 -> 852.2 mm
- net ROW0: track 687.5 -> 822.0 mm
- net COL11: track 232.8 -> 366.2 mm
- net COL1: track 933.3 -> 1065.0 mm
- net COL13: track 390.7 -> 515.2 mm
- net COL3: track 842.1 -> 965.8 mm
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Other:
- board text added: "The board is designed as a two-sided board. However, the historic board is one- sided. If there is no additional fabrication cost: * Copper only on the BACK side. Through-hole plating is not required anywhere. * Solder mask only on BACK side. * Silkscreen on BOTH sides."
- board text removed: "* Copper only on the BACK side. Through-hole plating is not required. * Solder mask only on BACK side. * Silkscreen only on the FRONT side."
