File: SpaceCadet.kicad_pcb (KiCad board)
At the start: 2 copper layers, 469 x 166.6 mm, 202 parts, among them J0 Conn_02x17_Odd_Even, J3_1 Conn_01x04, J3_2 Conn_01x04, SW1 SD_4B3E, SW10 SD_4B3E, SW100 SD_4B3E, SW101 SD_4B3E, SW102 SD_4B3E, SW103 SD_4B3E, SW104 SD_4B3E, SW105 SD_4B3E, SW106 SD_4B3E, SW107 SD_4B3E, SW108 SD_4B3E, SW109 SD_4B3E, SW11 SD_4B3E, SW110 SD_4B3E, SW111 SD_4B3E, SW112 SD_4B3E, SW113 SD_4B3E, SW114 SD_4B3E, SW115 SD_4B3E, SW116 SD_4B3E, SW117 SD_4B3E, SW118 SD_4B3E, SW119 SD_4B3E, SW12 SD_4B3E, SW120 SD_4B3E, SW121 SD_4B3E, SW122 SD_4B3E, SW122a0 SD_4B3E, SW123 SD_4B3E, SW123a0 SD_4B3E, SW124 SD_4B3E, SW124a0 SD_4B3E, SW125 SD_4B3E, SW126 SD_4B3E, SW127 SD_4B3E, SW128 SD_4B3E, SW13 SD_4B3E, SW14 SD_4B3E, SW15 SD_4B3E, SW16 SD_4B3E, SW17 SD_4B3E, SW18 SD_4B3E, SW19 SD_4B3E, SW2 SD_4B3E, SW20 SD_4B3E, SW21 SD_4B3E, SW22 SD_4B3E, SW23 SD_4B3E, SW24 SD_4B3E, SW25 SD_4B3E, SW26 SD_4B3E, SW27 SD_4B3E, SW28 SD_4B3E, SW29 SD_4B3E, SW3 SD_4B3E, SW30 SD_4B3E, SW31 SD_4B3E, SW32 SD_4B3E, SW33 SD_4B3E, SW34 SD_4B3E, SW35 SD_4B3E, SW36 SD_4B3E, SW37 SD_4B3E, SW38 SD_4B3E, SW39 SD_4B3E, SW4 SD_4B3E, SW40 SD_4B3E, SW41 SD_4B3E, SW42 SD_4B3E, SW43 SD_4B3E, SW44 SD_4B3E, SW45 SD_4B3E, SW46 SD_4B3E, SW47 SD_4B3E, SW48 SD_4B3E, SW49 SD_4B3E, SW5 SD_4B3E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

Commit message: Entered correct values for pom pom switches and some others.
Parts:
- SW1, SW112, SW12, SW14, SW16, SW18, SW20, SW22, SW24, SW27, SW3, SW46, SW5, SW52, SW69, SW7, SW72, SW74, SW9, SW92, SW94, SW99: value SD_4B3E -> SD_6B1D
- SW10, SW11, SW13, SW15, SW17, SW19, SW2, SW21, SW23, SW4, SW6, SW8: value SD_4B3E -> SD_4B1E
- SW115, SW119, SW122a0, SW123a0, SW124, SW127, SW41, SW89, SW97: value SD_4B3E -> UNPOPULATED
- SW73, SW95: value SD_4B3E -> SD_5B3E

Commit message: Corrections.
Parts:
- SW117, SW76: value SD_4B3E -> SD_5B3E
