File: Switch Matrix.kicad_sch (KiCad schematic)
At the start: 131 parts, among them SW1 SD_4B3E, SW10 SD_4B3E, SW100 SD_4B3E, SW101 SD_4B3E, SW102 SD_4B3E, SW103 SD_4B3E, SW104 SD_4B3E, SW105 SD_4B3E, SW106 SD_4B3E, SW107 SD_4B3E, SW108 SD_4B3E, SW109 SD_4B3E, SW11 SD_4B3E, SW110 SD_4B3E, SW111 SD_4B3E, SW112 SD_4B3E, SW113 SD_4B3E, SW114 SD_4B3E, SW115 SD_4B3E, SW116 SD_4B3E, SW117 SD_4B3E, SW118 SD_4B3E, SW119 SD_4B3E, SW12 SD_4B3E, SW120 SD_4B3E, SW121 SD_4B3E, SW122 SD_4B3E, SW122a0 SD_4B3E, SW123 SD_4B3E, SW123a0 SD_4B3E, SW124 SD_4B3E, SW124a0 SD_4B3E, SW125 SD_4B3E, SW126 SD_4B3E, SW127 SD_4B3E, SW128 SD_4B3E, SW13 SD_4B3E, SW14 SD_4B3E, SW15 SD_4B3E, SW16 SD_4B3E, SW17 SD_4B3E, SW18 SD_4B3E, SW19 SD_4B3E, SW2 SD_4B3E, SW20 SD_4B3E, SW21 SD_4B3E, SW22 SD_4B3E, SW23 SD_4B3E, SW24 SD_4B3E, SW25 SD_4B3E, SW26 SD_4B3E, SW27 SD_4B3E, SW28 SD_4B3E, SW29 SD_4B3E, SW3 SD_4B3E, SW30 SD_4B3E, SW31 SD_4B3E, SW32 SD_4B3E, SW33 SD_4B3E, SW34 SD_4B3E, SW35 SD_4B3E, SW36 SD_4B3E, SW37 SD_4B3E, SW38 SD_4B3E, SW39 SD_4B3E, SW4 SD_4B3E, SW40 SD_4B3E, SW41 SD_4B3E, SW42 SD_4B3E, SW43 SD_4B3E, SW44 SD_4B3E, SW45 SD_4B3E, SW46 SD_4B3E, SW47 SD_4B3E, SW48 SD_4B3E, SW49 SD_4B3E, SW5 SD_4B3E, SW50 SD_4B3E, SW51 SD_4B3E, SW52 SD_4B3E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

Commit message: Modern EDA route, initial commit.
Connections:
- net COL0: now also SW120.3 (VOUT), SW22.3 (VOUT), SW3.3 (VOUT), SW46.3 (VOUT), SW73.3 (VOUT), SW97.3 (VOUT); no longer SW119.3 (VOUT), SW23.3 (VOUT), SW47.3 (VOUT), SW72.3 (VOUT), SW96.3 (VOUT)
- net COL1: now also SW119.3 (VOUT), SW2.3 (VOUT), SW23.3 (VOUT), SW47.3 (VOUT), SW72.3 (VOUT), SW96.3 (VOUT); no longer SW120.3 (VOUT), SW22.3 (VOUT), SW46.3 (VOUT), SW73.3 (VOUT), SW97.3 (VOUT)
- net GND renamed +5V
- net +5V: no longer SW122a0.2 (GND), SW123a0.2 (GND), SW124a0.2 (GND)
Other:
- moved on the sheet: SW119, SW120, SW22, SW23, SW46, SW47, SW72, SW73, SW96, SW97

Commit message: Now one-sided board.
Connections:
- net +5V: now also SW122a0.2 (+5V), SW123a0.2 (+5V), SW124a0.2 (+5V)
Other:
- note added: "Dummy stabilizer switches are installed in these switches (designators with a0 suffix) despite being connected as normal switches in circuit. They have the same position (row & column) in the switch matrix as their non-suffixed counterparts."
- note added: "Switch Matrix"
Changed lines of the file:
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@@
   (junction (at 129.54 107.95) (diameter 0) (color 0 0 0 0)
   )
+  (junction (at 124.46 256.54) (diameter 0) (color 0 0 0 0)
+  )
   (junction (at 179.07 81.28) (diameter 0) (color 0 0 0 0)
   )
@@
   (junction (at 245.11 172.72) (diameter 0) (color 0 0 0 0)
   )
+  (junction (at 147.32 256.54) (diameter 0) (color 0 0 0 0)
+  )
   (junction (at 157.48 69.85) (diameter 0) (color 0 0 0 0)
   )
@@
     (stroke (width 0) (type default) (color 132 132 132 1))
   )
-  (wire (pts (xy 337.82 34.29) (xy 337.82 58.42))
-    (stroke (width 0) (type default) (color 0 0 0 0))
-  )
   (wire (pts (xy 283.21 172.72) (xy 295.91 172.72))
     (stroke (width 0) (type default) (color 132 132 132 1))
@@
     (stroke (width 0) (type default) (color 132 132 132 1))
   )
+  (wire (pts (xy 147.32 256.54) (xy 124.46 256.54))
+    (stroke (width 0) (type default) (color 0 0 0 0))
+  )
   (wire (pts (xy 171.45 88.9) (xy 171.45 107.95))
     (stroke (width 0) (type default) (color 0 0 0 0))
@@
     (stroke (width 0) (type default) (color 0 0 0 0))
   )
+  (wire (pts (xy 171.45 256.54) (xy 147.32 256.54))
+    (stroke (width 0) (type default) (color 0 0 0 0))
+  )
   (wire (pts (xy 115.57 69.85) (xy 115.57 88.9))
     (stroke (width 0) (type default) (color 0 0 0 0))
@@
     (stroke (width 0) (type default) (color 132 132 132 1))
   )
+  (wire (pts (xy 337.82 43.18) (xy 337.82 58.42))
+    (stroke (width 0) (type default) (color 132 132 132 1))
+  )
   (wire (pts (xy 109.22 100.33) (xy 123.19 100.33))
     (stroke (width 0) (type default) (color 255 0 0 1))
@@
     (stroke (width 0) (type default) (color 0 0 0 0))
   )
+  (wire (pts (xy 113.03 236.22) (xy 113.03 256.54))
+    (stroke (width 0) (type default) (color 0 0 0 0))
+  )
+  (wire (pts (xy 124.46 256.54) (xy 113.03 256.54))
+    (stroke (width 0) (type default) (color 0 0 0 0))
+  )
   (wire (pts (xy 337.82 77.47) (xy 337.82 96.52))
     (stroke (width 0) (type default) (color 132 132 132 1))
@@
   (wire (pts (xy 295.91 58.42) (xy 308.61 58.42))
     (stroke (width 0) (type default) (color 132 132 132 1))
+  )
+  (text "Switch Matrix" (at 86.995 31.75 0)
+    (effects (font (size 2.54 2.54)) (justify left bottom))
+  )
+  (text "Dummy stabilizer switches are installed in these switches (designators \nwith a0 suffix) despite being connected as normal switches in circuit. \nThey have the same position (row & column) in the switch matrix as \ntheir non-suffixed counterparts."
+    (at 113.03 266.7 0)
+    (effects (font (size 1.27 1.27)) (justify left bottom))
   )
   (global_label "ROW2" (shape input) (at 95.25 81.28 180) (fields_autoplaced)
@@
     (pin "3")
   )
+  (symbol (lib_id "power:+5V") (at 113.03 236.22 0) (unit 1)
+    (in_bom yes) (on_board yes) (fields_autoplaced)
+    (property "Reference" "#PWR0114" (id 0) (at 113.03 240.03 0)
+      (effects (font (size 1.27 1.27)) hide)
+    )
+    (property "Value" "+5V" (id 1) (at 113.03 232.6442 0))
+    (property "Footprint" "" (id 2) (at 113.03 236.22 0)
+      (effects (font (size 1.27 1.27)) hide)
+    )
+    (property "Datasheet" "" (id 3) (at 113.03 236.22 0)
+      (effects (font (size 1.27 1.27)) hide)
+    )
+    (pin "1")
+  )
   (symbol (lib_name "SD_4B3E_39") (lib_id "MicroSwitch_SD_4B3E:SD_4B3E") (at 308.61 107.95 0) (unit 1)
     (in_bom yes) (on_board yes)
@@
     (pin "3")
   )
-  (symbol (lib_id "power:+5V") (at 337.82 34.29 0) (unit 1)
+  (symbol (lib_id "power:+5V") (at 337.82 43.18 0) (unit 1)
     (in_bom yes) (on_board yes) (fields_autoplaced)
-    (property "Reference" "#PWR0113" (id 0) (at 337.82 38.1 0)
-      (effects (font (size 1.27 1.27)) hide)
-    )
-    (property "Value" "+5V" (id 1) (at 337.82 30.7142 0))
-    (property "Footprint" "" (id 2) (at 337.82 34.29 0)
-      (effects (font (size 1.27 1.27)) hide)
-    )
-    (property "Datasheet" "" (id 3) (at 337.82 34.29 0)
-      (effects (font (size 1.27 1.27)) hide)
-    )
+    (property "Reference" "#PWR0113" (id 0) (at 337.82 46.99 0)
+      (effects (font (size 1.27 1.27)) hide)
+    )
+    (property "Value" "+5V" (id 1) (at 337.82 39.6042 0))
+    (property "Footprint" "" (id 2) (at 337.82 43.18 0)
+      (effects (font (size 1.27 1.27)) hide)
+    )
+    (property "Datasheet" "" (id 3) (at 337.82 43.18 0)
+      (effects (font (size 1.27 1.27)) hide)
+    )

Commit message: Corrections.
Parts:
- SW1, SW112, SW12, SW14, SW16, SW18, SW20, SW22, SW24, SW27, SW3, SW46, SW5, SW52, SW69, SW7, SW72, SW74, SW9, SW92, SW94, SW99: value SD_4B3E -> SD_6B1D
- SW10, SW11, SW13, SW15, SW17, SW19, SW2, SW21, SW23, SW4, SW6, SW8: value SD_4B3E -> SD_4B1E
- SW115, SW119, SW122a0, SW123a0, SW127, SW41, SW89, SW97: value SD_4B3E -> UNPOPULATED
- SW117, SW73, SW76, SW95: value SD_4B3E -> SD_5B3E
- SW124: value SD_4B3E -> UNPOPULATED; Notes (none) -> Plastic stabilizer bracket inhabits this position.
